File: air/osd/hardware/64_pin_lite/expansion.sch (KiCad schematic (older format))
At the start: 5 parts, among them P2 CONN_20, P3 CONN_20

Commit message: sasve before moving psu caps on osd
Parts:
- C39: value C -> 10uF
- R30: value R -> 9K
- R31: value R -> 3K
Other:
- note added: "3V max"
Changed lines of the file:
@@
-EESchema Schematic File Version 2  date Wed 03 Dec 2014 09:37:23 GMT
+EESchema Schematic File Version 2  date Sun 07 Dec 2014 14:25:55 GMT
 LIBS:power
 LIBS:device
@@
 Sheet 5 8
 Title ""
-Date "3 dec 2014"
+Date "7 dec 2014"
 Rev ""
 Comp ""
@@
 Comment4 ""
 $EndDescr
+Text Notes 5550 3550 0    45   ~ 0
+3V max
 Connection ~ 4650 3400
 Wire Wire Line
@@
 P 5550 4000
 F 0 "C39" H 5600 4100 50  0000 L CNN
-F 1 "C" H 5600 3900 50  0000 L CNN
+F 1 "10uF" H 5600 3900 50  0000 L CNN
 	1    5550 4000
 	1    0    0    -1
@@
 P 5300 3950
 F 0 "R31" V 5380 3950 50  0000 C CNN
-F 1 "R" V 5300 3950 50  0000 C CNN
+F 1 "3K" V 5300 3950 50  0000 C CNN
 	1    5300 3950
 	1    0    0    -1
@@
 P 5300 3300
 F 0 "R30" V 5380 3300 50  0000 C CNN
-F 1 "R" V 5300 3300 50  0000 C CNN
+F 1 "9K" V 5300 3300 50  0000 C CNN
 	1    5300 3300
 	1    0    0    -1
