File: air/osd/hardware/64_pin_lite/mcu.sch (KiCad schematic (older format))
At the start: 24 parts, among them P1 CONN_2, U1 SI501, U2 STM32F405RGT6, U3 74LVC1G86

Commit message: added links for isolted port and other mods
Changed lines of the file:
@@
-EESchema Schematic File Version 2  date Sun 30 Nov 2014 15:34:12 GMT
+EESchema Schematic File Version 2  date Mon 01 Dec 2014 08:28:41 GMT
 LIBS:power
 LIBS:device
@@
 Sheet 2 8
 Title ""
-Date "30 nov 2014"
+Date "1 dec 2014"
 Rev ""
 Comp ""
@@
 Text Label 2650 2825 2    45   ~ 0
 FRSKY_TXO_SIGN
-Text Notes 4975 1525 1    45   ~ 0
+Text Notes 5000 2850 1    45   ~ 0
 TIM3_ETR
 Text Notes 5575 2900 1    45   ~ 0

Commit message: on pcb added battery level resistor divider. On code compiled and built ok but not uploaded or tested
Other:
- note added: "ADC1 (Batt level)"
- note removed: "ADC1"
Changed lines of the file:
@@
-EESchema Schematic File Version 2  date Tue 02 Dec 2014 12:33:04 GMT
+EESchema Schematic File Version 2  date Wed 03 Dec 2014 09:37:23 GMT
 LIBS:power
 LIBS:device
@@
 Sheet 2 8
 Title ""
-Date "2 dec 2014"
+Date "3 dec 2014"
 Rev ""
 Comp ""
@@
 Text HLabel 4950 5625 3    45   BiDi ~ 0
 MCU_PB1
-Text Notes 5000 6225 1    45   ~ 0
-ADC1
+Text Notes 4975 6600 1    45   ~ 0
+ADC1 (Batt level)
 Text HLabel 4650 5625 3    45   BiDi ~ 0
 MCU_PC5

Commit message: sasve before moving psu caps on osd
Parts:
- added P6, P7, P8: CONN_1, symbol CONN_1
- D1: footprint (none) -> 0603
- U3: footprint (none) -> SOT23-5
Connections:
- net AV_TELEM_RXI: now also P7.1
- net AV_TELEM_TXO: now also P8.1
- net PIXEL_CLK: now also P6.1

Commit message: must be nearly finalised pcb ready for sending off.Disco circuit tested  so now just hope its right for pcb
Parts:
- L1: value Ferrite Bead -> 22nH
Changed lines of the file:
@@
-EESchema Schematic File Version 2  date Sun 07 Dec 2014 14:25:55 GMT
+EESchema Schematic File Version 2  date Sun 07 Dec 2014 19:48:20 GMT
 LIBS:power
 LIBS:device
@@
 P 2050 6050
 F 0 "L1" V 2000 6050 40  0000 C CNN
-F 1 "Ferrite Bead" V 2150 6050 40  0000 C CNN
+F 1 "22nH" V 2150 6050 40  0000 C CNN
 	1    2050 6050
 	0    1    1    0
