File: air/osd/hardware/64_pin_lite/camera.sch (KiCad schematic (older format))
At the start: 2 parts, among them K1 CONN_3

Commit message: removed traces on pcb design. Added links to separate ground paths for modules. Moved mpu to other side of board. Added 2 pin power conector at end of board
Parts:
- added LK15: LINK, symbol LINK
Connections:
- net labels added: VIN+
- wire segments 4 -> 7
Changed lines of the file:
@@
-EESchema Schematic File Version 2  date Mon 26 Jan 2015 12:32:55 GMT
+EESchema Schematic File Version 2  date Wed 04 Mar 2015 21:55:30 GMT
 LIBS:lm358
 LIBS:conn_6
@@
 LIBS:tlv3501
 LIBS:74lvc1g86
+LIBS:R0link
+LIBS:osd-cache
 EELAYER 25  0
 EELAYER END
@@
 Sheet 4 8
 Title ""
-Date "26 jan 2015"
+Date "4 mar 2015"
 Rev ""
 Comp ""
@@
 Comment4 ""
 $EndDescr
+Connection ~ 3900 3450
+Wire Wire Line
+	3900 3350 3900 3450
 Wire Wire Line
 	4100 3450 3750 3450
@@
 Wire Wire Line
 	4500 3450 5200 3450
+Wire Wire Line
+	3650 2750 3900 2750
+Wire Wire Line
+	3900 2750 3900 2850
+Text HLabel 3650 2750 0    45   Input ~ 0
+VIN+
+$Comp
+L LINK LK15
+U 1 1 54F752A1
+P 3900 3100
+F 0 "LK15" V 3980 3100 50  0000 C CNN
+F 1 "LINK" V 3900 3100 50  0000 C CNN
+	1    3900 3100
+	1    0    0    -1
+$EndComp
 $Comp
 L DIODESCH D4

Commit message: laid out components on boar. No traces done yet
Parts:
- removed LK15: LINK, symbol LINK
Connections:
- net labels removed: VIN+
- wire segments 7 -> 4
Changed lines of the file:
@@
-EESchema Schematic File Version 2  date Wed 04 Mar 2015 21:55:30 GMT
+EESchema Schematic File Version 2  date Thu 05 Mar 2015 23:13:03 GMT
 LIBS:lm358
 LIBS:conn_6
@@
 Sheet 4 8
 Title ""
-Date "4 mar 2015"
+Date "5 mar 2015"
 Rev ""
 Comp ""
@@
 Comment4 ""
 $EndDescr
-Connection ~ 3900 3450
-Wire Wire Line
-	3900 3350 3900 3450
 Wire Wire Line
 	4100 3450 3750 3450
@@
 Wire Wire Line
 	4500 3450 5200 3450
-Wire Wire Line
-	3650 2750 3900 2750
-Wire Wire Line
-	3900 2750 3900 2850
-Text HLabel 3650 2750 0    45   Input ~ 0
-VIN+
-$Comp
-L LINK LK15
-U 1 1 54F752A1
-P 3900 3100
-F 0 "LK15" V 3980 3100 50  0000 C CNN
-F 1 "LINK" V 3900 3100 50  0000 C CNN
-	1    3900 3100
-	1    0    0    -1
-$EndComp
 $Comp
 L DIODESCH D4
