File: air/osd/hardware/64_pin_lite/video_out.sch (KiCad schematic (older format))
At the start: 6 parts, among them P5 CONN_5, U7 LM358

Commit message: removed traces on pcb design. Added links to separate ground paths for modules. Moved mpu to other side of board. Added 2 pin power conector at end of board
Parts:
- added LK16: LINK, symbol LINK
Connections:
- net labels added: VIN+
- wire segments 28 -> 31
Other:
- moved on the sheet: P5
Changed lines of the file:
@@
-EESchema Schematic File Version 2  date Mon 26 Jan 2015 12:32:55 GMT
+EESchema Schematic File Version 2  date Wed 04 Mar 2015 21:55:31 GMT
 LIBS:lm358
 LIBS:conn_6
@@
 LIBS:tlv3501
 LIBS:74lvc1g86
+LIBS:R0link
+LIBS:osd-cache
 EELAYER 25  0
 EELAYER END
@@
 Sheet 7 8
 Title ""
-Date "26 jan 2015"
+Date "4 mar 2015"
 Rev ""
 Comp ""
@@
 $EndDescr
 Wire Wire Line
+	7100 3350 7100 3500
+Wire Wire Line
+	7100 3500 6900 3500
+Wire Wire Line
 	5150 2350 4950 2350
 Connection ~ 3150 4900
@@
 Wire Wire Line
 	8550 2350 5550 2350
+Wire Wire Line
+	7100 2850 7100 2650
+Connection ~ 7100 2650
+Text HLabel 6900 3500 0    45   Input ~ 0
+VIN+
+$Comp
+L LINK LK16
+U 1 1 54F752D2
+P 7100 3100
+F 0 "LK16" V 7180 3100 50  0000 C CNN
+F 1 "LINK" V 7100 3100 50  0000 C CNN
+	1    7100 3100
+	1    0    0    -1
+$EndComp
 $Comp
 L C C25
@@
 L CONN_5 P5
 U 1 1 546DBC86
-P 8900 2550
-F 0 "P5" V 8850 2550 50  0000 C CNN
-F 1 "CONN_5" V 8950 2550 50  0000 C CNN
-	1    8900 2550
+P 8950 2550
+F 0 "P5" V 8900 2550 50  0000 C CNN
+F 1 "CONN_5" V 9000 2550 50  0000 C CNN
+	1    8950 2550
 	1    0    0    1
 $EndComp

Commit message: laid out components on boar. No traces done yet
Parts:
- removed LK16: LINK, symbol LINK
Connections:
- net labels added: BUF_DAC_OUT1, BUF_DAC_OUT2, LINE_DAC_OUT1, LINE_DAC_OUT2
- net labels removed: VIN+
- wire segments 31 -> 28
Changed lines of the file:
@@
-EESchema Schematic File Version 2  date Wed 04 Mar 2015 21:55:31 GMT
+EESchema Schematic File Version 2  date Thu 05 Mar 2015 23:13:03 GMT
 LIBS:lm358
 LIBS:conn_6
@@
 Sheet 7 8
 Title ""
-Date "4 mar 2015"
+Date "5 mar 2015"
 Rev ""
 Comp ""
@@
 Comment4 ""
 $EndDescr
-Wire Wire Line
-	7100 3350 7100 3500
-Wire Wire Line
-	7100 3500 6900 3500
+Text Label 6000 3550 0    45   ~ 0
+LINE_DAC_OUT2
+Text Label 6000 2350 0    45   ~ 0
+LINE_DAC_OUT1
+Text Label 4800 4050 0    45   ~ 0
+BUF_DAC_OUT2
+Text Label 4800 2900 0    45   ~ 0
+BUF_DAC_OUT1
 Wire Wire Line
 	5150 2350 4950 2350
@@
 Wire Wire Line
 	8550 2350 5550 2350
-Wire Wire Line
-	7100 2850 7100 2650
-Connection ~ 7100 2650
-Text HLabel 6900 3500 0    45   Input ~ 0
-VIN+
-$Comp
-L LINK LK16
-U 1 1 54F752D2
-P 7100 3100
-F 0 "LK16" V 7180 3100 50  0000 C CNN
-F 1 "LINK" V 7100 3100 50  0000 C CNN
-	1    7100 3100
-	1    0    0    -1
-$EndComp
 $Comp
 L C C25
