File: air/osd/hardware/64_pin_lite/video_out.sch (KiCad schematic (older format))
At the start: 6 parts, among them P5 CONN_5, U7 LM358

Commit message: added some 3 terminal EMI filters to the board
Parts:
- added C45: 0u1, symbol C
- added FI3: NFL18ST207X1C3, symbol EMI_FILTER3
Connections:
- wire segments 28 -> 34
Other:
- moved on the sheet: D5, P5
Changed lines of the file:
@@
-EESchema Schematic File Version 2  date Thu 12 Mar 2015 15:44:15 GMT
+EESchema Schematic File Version 2  date Wed 17 Jun 2015 00:34:32 BST
 LIBS:lm358
 LIBS:conn_6
@@
 LIBS:74lvc1g86
 LIBS:R0link
+LIBS:emi_filter
 LIBS:osd-cache
 EELAYER 25  0
@@
 Sheet 7 8
 Title ""
-Date "12 mar 2015"
+Date "16 jun 2015"
 Rev ""
 Comp ""
@@
 Comment4 ""
 $EndDescr
-Text Label 6000 3550 0    45   ~ 0
+Connection ~ 7750 3550
+Wire Wire Line
+	7750 2800 7750 3550
+Wire Wire Line
+	7050 3150 7050 3550
+Wire Wire Line
+	7050 3550 9000 3550
+Connection ~ 9000 2750
+Wire Wire Line
+	9000 3550 9000 2750
+Wire Wire Line
+	9100 2350 5550 2350
+Connection ~ 3150 5950
+Wire Wire Line
+	4150 5600 4150 5950
+Wire Wire Line
+	4150 5950 3100 5950
+Wire Wire Line
+	3150 4950 3150 4900
+Wire Wire Line
+	8950 2750 9100 2750
+Wire Wire Line
+	9100 2550 8900 2550
+Wire Wire Line
+	9100 2450 5750 2450
+Wire Wire Line
+	5750 2450 5750 3600
+Wire Wire Line
+	5750 3600 5600 3600
+Wire Wire Line
+	4700 3600 5200 3600
+Wire Wire Line
+	3700 3500 3300 3500
+Wire Wire Line
+	4700 2400 4950 2400
+Wire Wire Line
+	3400 2300 3700 2300
+Wire Wire Line
+	3700 2500 3550 2500
+Wire Wire Line
+	3550 2500 3550 2900
+Wire Wire Line
+	3550 2900 4800 2900
+Wire Wire Line
+	4800 2900 4800 2400
+Connection ~ 4800 2400
+Wire Wire Line
+	3700 3700 3600 3700
+Wire Wire Line
+	3600 3700 3600 4050
+Wire Wire Line
+	3600 4050 4800 4050
+Wire Wire Line
+	4800 4050 4800 3600
+Connection ~ 4800 3600
+Wire Wire Line
+	4950 2400 4950 2350
+Wire Wire Line
+	6450 2650 6350 2650
+Wire Wire Line
+	9100 2650 8050 2650
+Wire Wire Line
+	6850 2650 7450 2650
+Wire Wire Line
+	3150 5850 3150 5950
+Wire Wire Line
+	3050 4900 4150 4900
+Wire Wire Line
+	4150 4900 4150 5200
+Connection ~ 3150 4900
+Wire Wire Line
+	4950 2350 5150 2350
+Wire Wire Line
+	7050 2750 7050 2650
+Connection ~ 7050 2650
+$Comp
+L EMI_FILTER3 FI3
+U 1 1 5580B15C
+P 7750 2650
+F 0 "FI3" H 7900 2800 60  0000 C CNN
+F 1 "NFL18ST207X1C3" H 8150 2400 60  0000 C CNN
+	1    7750 2650
+	1    0    0    -1
+$EndComp
+$Comp
+L C C45
+U 1 1 5580B0E2
+P 7050 2950
+F 0 "C45" H 7100 3050 50  0000 L CNN
+F 1 "0u1" H 7100 2850 50  0000 L CNN
+	1    7050 2950
+	1    0    0    -1
+$EndComp
+Text Label 5700 3600 0    45   ~ 0
 LINE_DAC_OUT2
 Text Label 6000 2350 0    45   ~ 0
@@
 Text Label 4800 2900 0    45   ~ 0
 BUF_DAC_OUT1
-Wire Wire Line
-	5150 2350 4950 2350
-Connection ~ 3150 4900
-Wire Wire Line
-	4150 5200 4150 4900
-Wire Wire Line
-	4150 4900 3050 4900
-Wire Wire Line
-	3150 5850 3150 5950
-Wire Wire Line
-	8550 2650 7600 2650
-Wire Wire Line
-	7200 2650 7000 2650
-Wire Wire Line
-	4950 2350 4950 2400
-Connection ~ 4800 3600
-Wire Wire Line
-	4800 3600 4800 4050
-Wire Wire Line
-	4800 4050 3600 4050
-Wire Wire Line
-	3600 4050 3600 3700
-Wire Wire Line
-	3600 3700 3700 3700
-Connection ~ 4800 2400
-Wire Wire Line
-	4800 2400 4800 2900
-Wire Wire Line
-	4800 2900 3550 2900
-Wire Wire Line
-	3550 2900 3550 2500
-Wire Wire Line
-	3550 2500 3700 2500
-Wire Wire Line
-	3400 2300 3700 2300
-Wire Wire Line
-	4950 2400 4700 2400
-Wire Wire Line
-	3700 3500 3300 3500
-Wire Wire Line
-	4700 3600 5200 3600
-Wire Wire Line
-	5600 3600 6000 3600
-Wire Wire Line
-	6000 3600 6000 2450
-Wire Wire Line
-	6000 2450 8550 2450
-Wire Wire Line
-	8550 2550 8250 2550
-Wire Wire Line
-	8550 2750 8350 2750
-Wire Wire Line
-	3150 4900 3150 4950
-Wire Wire Line
-	3100 5950 4150 5950
-Wire Wire Line
-	4150 5950 4150 5600
-Connection ~ 3150 5950
-Wire Wire Line
-	8550 2350 5550 2350
 $Comp
 L C C25
@@
 L DIODESCH D5
 U 1 1 546F5AD9
-P 7400 2650
-F 0 "D5" H 7400 2750 40  0000 C CNN
-F 1 "DIODESCH" H 7400 2550 40  0000 C CNN
-	1    7400 2650
+P 6650 2650
+F 0 "D5" H 6650 2750 40  0000 C CNN
+F 1 "DIODESCH" H 6650 2550 40  0000 C CNN
+	1    6650 2650
 	1    0    0    -1
 $EndComp
 Text HLabel 3400 2300 0    60   Input ~ 0
 RAW_DAC_OUT1
-Text HLabel 7000 2650 0    45   Input ~ 0
+Text HLabel 6350 2650 0    45   Input ~ 0
 VIDEO_OUT_+V
-Text HLabel 8350 2750 0    45   BiDi ~ 0
+Text HLabel 8950 2750 0    45   BiDi ~ 0
 VIDEO_OUT_GND
 $Comp
 L CONN_5 P5
 U 1 1 546DBC86
-P 8950 2550
-F 0 "P5" V 8900 2550 50  0000 C CNN
-F 1 "CONN_5" V 9000 2550 50  0000 C CNN
-	1    8950 2550
+P 9500 2550
+F 0 "P5" V 9450 2550 50  0000 C CNN
+F 1 "CONN_5" V 9550 2550 50  0000 C CNN
+	1    9500 2550
 	1    0    0    1
 $EndComp
-Text HLabel 8250 2550 0    45   Input ~ 0
+Text HLabel 8900 2550 0    45   Input ~ 0
 VIDEO_OUT
 $Comp
