File: air/osd/hardware/64_pin_lite/video_io_FMS6141_sync_clamp.sch (KiCad schematic (older format))
At the start: 33 parts, among them P10 CONN_1, P12 CONN_1, P9 CONN_1, U10 FMS6141, U11 DAC084S085, U12 ADG704, U13 OPA830, U8 MCP6562, U9 TLV3501

Commit message: before trying 5v plane
Parts:
- added C44: 4U7, symbol CP1
Connections:
- net VIDEO_+5V: now also C44.1
- net VIDEO_GND: now also C44.2
Changed lines of the file:
@@
-EESchema Schematic File Version 2  date Mon 09 Mar 2015 16:29:56 GMT
+EESchema Schematic File Version 2  date Wed 11 Mar 2015 10:11:51 GMT
 LIBS:lm358
 LIBS:conn_6
@@
 Sheet 8 8
 Title ""
-Date "9 mar 2015"
+Date "11 mar 2015"
 Rev ""
 Comp ""
@@
 Comment4 ""
 $EndDescr
+Connection ~ 7600 6250
+Wire Wire Line
+	7600 5950 7600 6250
 Connection ~ 3300 700
 Wire Wire Line
-	3150 700  6100 700
+	3150 700  3300 700
+Wire Wire Line
+	3300 700  6100 700
 Connection ~ 5700 5900
 Wire Wire Line
@@
 	5700 1850 6250 1850
 Wire Wire Line
-	6450 5450 7250 5450
-Wire Wire Line
 	1250 6550 1550 6550
 Wire Wire Line
@@
 	2550 2050 2550 2850
 Wire Wire Line
-	2550 2850 1300 2850
+	2550 2850 1350 2850
+Wire Wire Line
+	1350 2850 1300 2850
 Wire Wire Line
 	2550 1150 2550 950
 Wire Wire Line
 	2550 950  2400 950
-Connection ~ 7650 6250
-Wire Wire Line
-	7650 6250 7650 6700
+Connection ~ 7850 6250
+Wire Wire Line
+	7850 6250 7850 6700
 Connection ~ 9600 5450
 Wire Wire Line
@@
 Connection ~ 6950 5450
 Wire Wire Line
-	6950 5550 6950 5450
+	6950 5450 6950 5550
 Connection ~ 7250 6250
 Wire Wire Line
@@
 	8400 6250 8400 5950
 Wire Wire Line
-	6650 6250 9900 6250
+	6650 6250 6950 6250
+Wire Wire Line
+	6950 6250 7250 6250
+Wire Wire Line
+	7250 6250 7600 6250
+Wire Wire Line
+	7600 6250 7850 6250
+Wire Wire Line
+	7850 6250 8400 6250
+Wire Wire Line
+	8400 6250 8700 6250
+Wire Wire Line
+	8700 6250 9000 6250
+Wire Wire Line
+	9000 6250 9300 6250
+Wire Wire Line
+	9300 6250 9600 6250
+Wire Wire Line
+	9600 6250 9900 6250
 Wire Wire Line
 	9900 6250 9900 5950
@@
 	2900 4100 3200 4100
 Wire Wire Line
-	5600 6400 5800 6400
+	5800 6400 5700 6400
+Wire Wire Line
+	5700 6400 5600 6400
 Connection ~ 10000 1600
 Wire Wire Line
@@
 	8900 2400 8900 1700
 Wire Wire Line
-	1500 1600 1250 1600
+	1250 1600 1350 1600
+Wire Wire Line
+	1350 1600 1500 1600
 Connection ~ 3300 1600
 Wire Wire Line
@@
 Connection ~ 5700 6400
 Wire Wire Line
-	5700 6400 5700 5550
+	5700 6400 5700 5900
+Wire Wire Line
+	5700 5900 5700 5550
 Wire Wire Line
 	5700 5550 5250 5550
@@
 	4200 7200 4200 7350
 Wire Wire Line
-	4200 7350 3650 7350
+	4200 7350 3950 7350
+Wire Wire Line
+	3950 7350 3650 7350
 Wire Wire Line
 	3650 7350 3650 6700
 Connection ~ 4200 6250
 Wire Wire Line
-	4200 6250 4600 6250
+	4600 6250 4400 6250
+Wire Wire Line
+	4400 6250 4200 6250
 Wire Wire Line
 	4600 6550 3900 6550
@@
 	3650 2350 3850 2350
 Wire Wire Line
-	4800 1200 4800 1000
+	4800 1000 4800 1100
+Wire Wire Line
+	4800 1100 4800 1200
 Wire Wire Line
 	6650 1400 6400 1400
@@
 	7650 2150 7800 2150
 Wire Wire Line
-	3300 700  3300 3100
+	3300 700  3300 1600
+Wire Wire Line
+	3300 1600 3300 3100
 Wire Wire Line
 	7350 2150 7350 3700
@@
 	1850 6350 1300 6350
 Wire Wire Line
-	1300 6350 1300 3100
+	1300 6350 1300 4900
+Wire Wire Line
+	1300 4900 1300 4250
+Wire Wire Line
+	1300 4250 1300 3100
 Wire Wire Line
 	3050 6200 2850 6200
 Wire Wire Line
-	3650 6300 3650 6200
+	3650 6200 3650 6300
 Connection ~ 3650 6200
 Wire Wire Line
-	4200 6050 4200 6700
-Wire Wire Line
-	3900 6200 3550 6200
+	4200 6700 4200 6250
+Wire Wire Line
+	4200 6250 4200 6050
+Wire Wire Line
+	3900 6200 3800 6200
+Wire Wire Line
+	3800 6200 3650 6200
+Wire Wire Line
+	3650 6200 3550 6200
 Wire Wire Line
 	4400 6250 4400 5550
@@
 Connection ~ 4400 6250
 Wire Wire Line
-	8700 1500 8950 1500
+	8950 1500 8800 1500
+Wire Wire Line
+	8800 1500 8700 1500
 Wire Wire Line
 	8800 2100 8800 2400
 Wire Wire Line
-	8800 2400 9200 2400
+	8800 2400 8900 2400
+Wire Wire Line
+	8900 2400 9200 2400
 Connection ~ 8900 2400
 Wire Wire Line
@@
 	1350 2400 1350 2850
 Wire Wire Line
-	10050 1600 9950 1600
+	9950 1600 10000 1600
+Wire Wire Line
+	10000 1600 10050 1600
 Wire Wire Line
 	1300 4250 1750 4250
 Connection ~ 1300 4250
 Wire Wire Line
-	6250 1200 6250 3500
+	6250 1200 6250 1850
+Wire Wire Line
+	6250 1850 6250 3500
 Wire Wire Line
 	4200 3500 4050 3500
@@
 	6250 3500 4700 3500
 Wire Wire Line
-	4050 3250 1600 3250
+	4050 3250 3200 3250
+Wire Wire Line
+	3200 3250 1600 3250
 Wire Wire Line
 	4050 3250 4050 3500
@@
 	2400 4700 2400 4500
 Wire Wire Line
-	3200 4500 3200 3900
+	3200 4500 3200 4100
+Wire Wire Line
+	3200 4100 3200 3900
 Connection ~ 3200 4100
 Wire Wire Line
-	8250 5450 9900 5450
+	8250 5450 8400 5450
+Wire Wire Line
+	8400 5450 8700 5450
+Wire Wire Line
+	8700 5450 9000 5450
+Wire Wire Line
+	9000 5450 9300 5450
+Wire Wire Line
+	9300 5450 9600 5450
+Wire Wire Line
+	9600 5450 9900 5450
 Wire Wire Line
 	8700 6250 8700 5950
@@
 Connection ~ 6650 5450
 Wire Wire Line
-	7250 5450 7250 5550
+	7250 5550 7250 5450
 Connection ~ 7250 5450
 Wire Wire Line
@@
 	9900 5450 9900 5550
 Wire Wire Line
-	7650 6700 7350 6700
+	7850 6700 7350 6700
 Connection ~ 1350 2850
 Wire Wire Line
@@
 Wire Wire Line
 	10550 1600 10600 1600
+Wire Wire Line
+	6450 5450 6650 5450
+Wire Wire Line
+	6650 5450 6950 5450
+Wire Wire Line
+	6950 5450 7250 5450
+Wire Wire Line
+	7250 5450 7600 5450
+Wire Wire Line
+	7600 5450 7600 5550
+$Comp
+L CP1 C44
+U 1 1 550014A9
+P 7600 5750
+F 0 "C44" H 7650 5850 50  0000 L CNN
+F 1 "4U7" H 7650 5650 50  0000 L CNN
+	1    7600 5750
+	1    0    0    -1
+$EndComp
 $Comp
 L CONN_1 P12

Commit message: hopefully finished
Changed lines of the file:
@@
-EESchema Schematic File Version 2  date Wed 11 Mar 2015 10:11:51 GMT
+EESchema Schematic File Version 2  date Wed 11 Mar 2015 17:51:25 GMT
 LIBS:lm358
 LIBS:conn_6
@@
 Connection ~ 7600 6250
 Wire Wire Line
-	7600 5950 7600 6250
+	7600 6250 7600 5950
 Connection ~ 3300 700
 Wire Wire Line
-	3150 700  3300 700
-Wire Wire Line
-	3300 700  6100 700
+	3150 700  6100 700
 Connection ~ 5700 5900
 Wire Wire Line
@@
 	2550 2050 2550 2850
 Wire Wire Line
-	2550 2850 1350 2850
-Wire Wire Line
-	1350 2850 1300 2850
+	2550 2850 1300 2850
 Wire Wire Line
 	2550 1150 2550 950
@@
 	8400 6250 8400 5950
 Wire Wire Line
-	6650 6250 6950 6250
-Wire Wire Line
-	6950 6250 7250 6250
-Wire Wire Line
-	7250 6250 7600 6250
-Wire Wire Line
-	7600 6250 7850 6250
-Wire Wire Line
-	7850 6250 8400 6250
-Wire Wire Line
-	8400 6250 8700 6250
-Wire Wire Line
-	8700 6250 9000 6250
-Wire Wire Line
-	9000 6250 9300 6250
-Wire Wire Line
-	9300 6250 9600 6250
-Wire Wire Line
-	9600 6250 9900 6250
+	6650 6250 9900 6250
 Wire Wire Line
 	9900 6250 9900 5950
@@
 	2900 4100 3200 4100
 Wire Wire Line
-	5800 6400 5700 6400
-Wire Wire Line
-	5700 6400 5600 6400
+	5800 6400 5600 6400
 Connection ~ 10000 1600
 Wire Wire Line
@@
 	8900 2400 8900 1700
 Wire Wire Line
-	1250 1600 1350 1600
-Wire Wire Line
-	1350 1600 1500 1600
+	1250 1600 1500 1600
 Connection ~ 3300 1600
 Wire Wire Line
@@
 Connection ~ 5700 6400
 Wire Wire Line
-	5700 6400 5700 5900
-Wire Wire Line
-	5700 5900 5700 5550
+	5700 6400 5700 5550
 Wire Wire Line
 	5700 5550 5250 5550
@@
 	4200 7200 4200 7350
 Wire Wire Line
-	4200 7350 3950 7350
-Wire Wire Line
-	3950 7350 3650 7350
+	4200 7350 3650 7350
 Wire Wire Line
 	3650 7350 3650 6700
 Connection ~ 4200 6250
 Wire Wire Line
-	4600 6250 4400 6250
-Wire Wire Line
-	4400 6250 4200 6250
+	4600 6250 4200 6250
 Wire Wire Line
 	4600 6550 3900 6550
@@
 	3650 2350 3850 2350
 Wire Wire Line
-	4800 1000 4800 1100
-Wire Wire Line
-	4800 1100 4800 1200
+	4800 1000 4800 1200
 Wire Wire Line
 	6650 1400 6400 1400
@@
 	7650 2150 7800 2150
 Wire Wire Line
-	3300 700  3300 1600
-Wire Wire Line
-	3300 1600 3300 3100
+	3300 700  3300 3100
 Wire Wire Line
 	7350 2150 7350 3700
@@
 	1850 6350 1300 6350
 Wire Wire Line
-	1300 6350 1300 4900
-Wire Wire Line
-	1300 4900 1300 4250
-Wire Wire Line
-	1300 4250 1300 3100
+	1300 6350 1300 3100
 Wire Wire Line
 	3050 6200 2850 6200
@@
 Connection ~ 3650 6200
 Wire Wire Line
-	4200 6700 4200 6250
-Wire Wire Line
-	4200 6250 4200 6050
-Wire Wire Line
-	3900 6200 3800 6200
-Wire Wire Line
-	3800 6200 3650 6200
-Wire Wire Line
-	3650 6200 3550 6200
+	4200 6700 4200 6050
+Wire Wire Line
+	3900 6200 3550 6200
 Wire Wire Line
 	4400 6250 4400 5550
@@
 Connection ~ 4400 6250
 Wire Wire Line
-	8950 1500 8800 1500
-Wire Wire Line
-	8800 1500 8700 1500
+	8950 1500 8700 1500
 Wire Wire Line
 	8800 2100 8800 2400
 Wire Wire Line
-	8800 2400 8900 2400
-Wire Wire Line
-	8900 2400 9200 2400
+	8800 2400 9200 2400
 Connection ~ 8900 2400
 Wire Wire Line
@@
 	1350 2400 1350 2850
 Wire Wire Line
-	9950 1600 10000 1600
-Wire Wire Line
-	10000 1600 10050 1600
+	9950 1600 10050 1600
 Wire Wire Line
 	1300 4250 1750 4250
 Connection ~ 1300 4250
 Wire Wire Line
-	6250 1200 6250 1850
-Wire Wire Line
-	6250 1850 6250 3500
+	6250 1200 6250 3500
 Wire Wire Line
 	4200 3500 4050 3500
@@
 	6250 3500 4700 3500
 Wire Wire Line
-	4050 3250 3200 3250
-Wire Wire Line
-	3200 3250 1600 3250
+	4050 3250 1600 3250
 Wire Wire Line
 	4050 3250 4050 3500
@@
 	2400 4700 2400 4500
 Wire Wire Line
-	3200 4500 3200 4100
-Wire Wire Line
-	3200 4100 3200 3900
+	3200 4500 3200 3900
 Connection ~ 3200 4100
 Wire Wire Line
-	8250 5450 8400 5450
-Wire Wire Line
-	8400 5450 8700 5450
-Wire Wire Line
-	8700 5450 9000 5450
-Wire Wire Line
-	9000 5450 9300 5450
-Wire Wire Line
-	9300 5450 9600 5450
-Wire Wire Line
-	9600 5450 9900 5450
+	8250 5450 9900 5450
 Wire Wire Line
 	8700 6250 8700 5950
@@
 Connection ~ 6650 5450
 Wire Wire Line
-	7250 5550 7250 5450
+	7250 5450 7250 5550
 Connection ~ 7250 5450
 Wire Wire Line
-	6650 5450 6650 5550
+	6650 5550 6650 5450
 Wire Wire Line
 	8700 5450 8700 5550
@@
 	10550 1600 10600 1600
 Wire Wire Line
-	6450 5450 6650 5450
-Wire Wire Line
-	6650 5450 6950 5450
-Wire Wire Line
-	6950 5450 7250 5450
-Wire Wire Line
-	7250 5450 7600 5450
+	6450 5450 7600 5450
 Wire Wire Line
 	7600 5450 7600 5550
