File: ground/tracker/v2/hardware/osd_v2_1_board.sch (KiCad schematic (older format))
At the start: 6 parts

Commit message: pan_motor servo initla draft aded, not tested yet
Connections:
- wire segments 34 -> 32
Changed lines of the file:
@@
-EESchema Schematic File Version 2  date Sat 16 May 2015 15:45:47 BST
+EESchema Schematic File Version 2  date Wed 20 May 2015 18:56:24 BST
 LIBS:quantracker
 LIBS:stm32
@@
 Sheet 3 3
 Title ""
-Date "16 may 2015"
+Date "20 may 2015"
 Rev ""
 Comp ""
@@
 	7000 4050 6700 4050
 Wire Wire Line
-	4750 3950 4450 3950
-Wire Wire Line
 	5850 4900 5850 4750
 Wire Wire Line
@@
 	4750 4250 4500 4250
 Wire Wire Line
-	4750 3450 4450 3450
+	4750 3450 4350 3450
 Wire Wire Line
 	4750 2950 4450 2950
@@
 	4750 3150 4450 3150
 Wire Wire Line
-	4750 3350 4450 3350
+	4750 3350 4300 3350
 Wire Wire Line
 	4750 4150 4500 4150
@@
 Wire Wire Line
 	5950 4900 5950 4750
-Wire Wire Line
-	4750 3850 4450 3850
 Wire Wire Line
 	4750 4050 4450 4050
@@
 Text Notes 3350 3600 2    60   ~ 0
 USART4-RXI/TIM5_CH2/ADC123_IN1
-Text Notes 3900 3500 2    60   ~ 0
+Text Notes 3500 3500 2    60   ~ 0
 ADC123_IN11\n
-Text Notes 3900 3400 2    60   ~ 0
+Text Notes 3500 3400 2    60   ~ 0
 ADC123_IN10\n
 Text Notes 3500 3000 2    60   ~ 0
@@
 Text HLabel 4450 4050 0    60   Input ~ 0
 VIDEO_RSSI
-Text HLabel 4450 3950 0    60   Input ~ 0
+Text HLabel 4350 3450 0    60   Input ~ 0
 MOTOR_CURRENT
-Text HLabel 4450 3850 0    60   Input ~ 0
+Text HLabel 4300 3350 0    60   Input ~ 0
 MOTOR_SPEED
 Text HLabel 7000 4050 2    60   Output ~ 0

Commit message: update ground V2 schematic
Parts:
- gave numbers to parts that had none: 6
Connections:
- net labels added: PAN_MOTOR_CURRENT, PAN_MOTOR_EMF
- net labels removed: MOTOR_CURRENT, MOTOR_SPEED
Changed lines of the file:
@@
-EESchema Schematic File Version 2  date Wed 20 May 2015 18:56:24 BST
+EESchema Schematic File Version 2  date Thu 21 May 2015 21:44:38 BST
 LIBS:quantracker
 LIBS:stm32
@@
 Sheet 3 3
 Title ""
-Date "20 may 2015"
+Date "21 may 2015"
 Rev ""
 Comp ""
@@
 PAN_SERVO_PWM
 $Comp
-L R R?
+L R R18
 U 1 1 55521193
 P 8150 1250
-F 0 "R?" V 8230 1250 50  0000 C CNN
+F 0 "R18" V 8230 1250 50  0000 C CNN
 F 1 "R" V 8150 1250 50  0000 C CNN
 	1    8150 1250
@@
 TILT_SERVO_PWM_RAW
 $Comp
-L R R?
+L R R17
 U 1 1 555210EC
 P 8100 1000
-F 0 "R?" V 8180 1000 50  0000 C CNN
+F 0 "R17" V 8180 1000 50  0000 C CNN
 F 1 "R" V 8100 1000 50  0000 C CNN
 	1    8100 1000
@@
 Video In
 $Comp
-L CONN_3 K?
+L CONN_3 K2
 U 1 1 55520FE6
 P 1850 6150
-F 0 "K?" V 1800 6150 50  0000 C CNN
+F 0 "K2" V 1800 6150 50  0000 C CNN
 F 1 "CONN_3" V 1900 6150 40  0000 C CNN
 	1    1850 6150
@@
 GPS
 $Comp
-L CONN_4 P?
+L CONN_4 P5
 U 1 1 55520E37
 P 1850 2550
-F 0 "P?" V 1800 2550 50  0000 C CNN
+F 0 "P5" V 1800 2550 50  0000 C CNN
 F 1 "CONN_4" V 1900 2550 50  0000 C CNN
 	1    1850 2550
@@
 Magnetometer
 $Comp
-L CONN_6 P?
+L CONN_6 P4
 U 1 1 55520DE1
 P 1850 1650
-F 0 "P?" V 1800 1650 60  0000 C CNN
+F 0 "P4" V 1800 1650 60  0000 C CNN
 F 1 "CONN_6" V 1900 1650 60  0000 C CNN
 	1    1850 1650
@@
 Text Notes 3350 3600 2    60   ~ 0
 USART4-RXI/TIM5_CH2/ADC123_IN1
-Text Notes 3500 3500 2    60   ~ 0
+Text Notes 3250 3500 2    60   ~ 0
 ADC123_IN11\n
-Text Notes 3500 3400 2    60   ~ 0
+Text Notes 3300 3400 2    60   ~ 0
 ADC123_IN10\n
 Text Notes 3500 3000 2    60   ~ 0
@@
 VIDEO_RSSI
 Text HLabel 4350 3450 0    60   Input ~ 0
-MOTOR_CURRENT
+PAN_MOTOR_CURRENT
 Text HLabel 4300 3350 0    60   Input ~ 0
-MOTOR_SPEED
+PAN_MOTOR_EMF
 Text HLabel 7000 4050 2    60   Output ~ 0
 LED3
@@
 PAN_MOTOR_DIR
 $Comp
-L OSD_V2_1 M?
+L OSD_V2_1 M1
 U 1 1 5551CEC6
 P 5700 3350
-F 0 "M?" H 5750 3100 60  0000 C CNN
+F 0 "M1" H 5750 3100 60  0000 C CNN
 F 1 "OSD_V2_1" H 5700 3350 60  0000 C CNN
 	1    5700 3350
