File: ground/tracker/v2/hardware/osd_v2_1_board.sch (KiCad schematic (older format))
At the start: 6 parts, among them K2 CONN_3, M1 OSD_V2_1, P4 CONN_6, P5 CONN_4

Commit message: added FreeCAD design files for V2 tracker
Connections:
- net labels added: MCU_GND, USART4_RXI, USART4_TXO
- net labels removed: PAN_MOTOR_QDRTA, PAN_MOTOR_QDRTB
- wire segments 32 -> 33
Changed lines of the file:
@@
-EESchema Schematic File Version 2  date Fri 29 May 2015 09:32:36 BST
+EESchema Schematic File Version 2  date Mon 01 Jun 2015 18:53:27 BST
 LIBS:quantracker
 LIBS:stm32
@@
 LIBS:tcm3105
 LIBS:quantracker_air_osd_v2_1
+LIBS:mc34931
 LIBS:tracker_using_quantracker_osd-cache
 EELAYER 25  0
@@
 $Descr A4 11700 8267
 encoding utf-8
-Sheet 3 3
+Sheet 4 4
 Title ""
-Date "28 may 2015"
+Date "1 jun 2015"
 Rev ""
 Comp ""
@@
 $EndDescr
 Wire Wire Line
+	4750 2550 4400 2550
+Wire Wire Line
+	6950 2950 6700 2950
+Wire Wire Line
+	4750 3550 4450 3550
+Wire Wire Line
+	7900 1250 7650 1250
+Wire Wire Line
+	6850 2650 6700 2650
+Wire Wire Line
+	4750 2850 4450 2850
+Wire Wire Line
+	7000 4250 6700 4250
+Wire Wire Line
+	4750 4050 4450 4050
+Wire Wire Line
+	5950 4900 5950 4750
+Wire Wire Line
+	5750 4900 5750 4750
+Wire Wire Line
+	7000 3750 6700 3750
+Wire Wire Line
+	7000 3450 6700 3450
+Wire Wire Line
+	7000 3250 6700 3250
+Wire Wire Line
+	4750 4150 4500 4150
+Wire Wire Line
+	4750 3350 4300 3350
+Wire Wire Line
+	4750 3150 4450 3150
+Wire Wire Line
+	4750 3050 4450 3050
+Wire Wire Line
+	6850 2750 6700 2750
+Wire Wire Line
+	4750 2950 4450 2950
+Wire Wire Line
+	4750 3450 4350 3450
+Wire Wire Line
+	4750 4250 4500 4250
+Wire Wire Line
+	7000 3350 6700 3350
+Wire Wire Line
+	7000 3650 6700 3650
+Wire Wire Line
+	5550 4900 5550 4750
+Wire Wire Line
+	5850 4900 5850 4750
+Wire Wire Line
+	7000 4050 6700 4050
+Wire Wire Line
+	7000 3850 6700 3850
+Wire Wire Line
+	7050 3950 6700 3950
+Wire Wire Line
+	8600 1000 8350 1000
+Wire Wire Line
+	7850 1000 7650 1000
+Wire Wire Line
+	8400 1250 8600 1250
+Wire Wire Line
+	4450 3650 4750 3650
+Wire Wire Line
 	6950 3050 6700 3050
-Wire Wire Line
-	4450 3650 4750 3650
-Wire Wire Line
-	8400 1250 8600 1250
-Wire Wire Line
-	7850 1000 7650 1000
-Wire Wire Line
-	8600 1000 8350 1000
-Wire Wire Line
-	7050 3950 6700 3950
-Wire Wire Line
-	7000 3850 6700 3850
-Wire Wire Line
-	7000 4050 6700 4050
-Wire Wire Line
-	5850 4900 5850 4750
-Wire Wire Line
-	5550 4900 5550 4750
-Wire Wire Line
-	7000 3650 6700 3650
-Wire Wire Line
-	7000 3350 6700 3350
-Wire Wire Line
-	4750 4250 4500 4250
-Wire Wire Line
-	4750 3450 4350 3450
-Wire Wire Line
-	4750 2950 4450 2950
-Wire Wire Line
-	6850 2750 6700 2750
-Wire Wire Line
-	4750 3050 4450 3050
-Wire Wire Line
-	4750 3150 4450 3150
-Wire Wire Line
-	4750 3350 4300 3350
-Wire Wire Line
-	4750 4150 4500 4150
-Wire Wire Line
-	7000 3250 6700 3250
-Wire Wire Line
-	7000 3450 6700 3450
-Wire Wire Line
-	7000 3750 6700 3750
-Wire Wire Line
-	5750 4900 5750 4750
-Wire Wire Line
-	5950 4900 5950 4750
-Wire Wire Line
-	4750 4050 4450 4050
-Wire Wire Line
-	7000 4250 6700 4250
-Wire Wire Line
-	4750 2850 4450 2850
-Wire Wire Line
-	6850 2650 6700 2650
-Wire Wire Line
-	7900 1250 7650 1250
-Wire Wire Line
-	4750 3550 4450 3550
-Wire Wire Line
-	6950 2950 6700 2950
+Text HLabel 4400 2550 0    60   Input ~ 0
+MCU_GND
 Text HLabel 6950 3050 2    60   Input ~ 0
 LCD_SCL
@@
 TILT_SERVO_PWM
 Text HLabel 4450 3550 0    60   Input ~ 0
-PAN_MOTOR_QDRTB
+USART4_RXI
 Text HLabel 4450 3650 0    60   Input ~ 0
-PAN_MOTOR_QDRTA
+USART4_TXO
 Text HLabel 4450 3150 0    60   Output ~ 0
 LED1

Commit message: moved pin setup to libs, cleaned up osd_example1 makefie to use osd,osd.hpp, added some docs
Parts:
- removed P4: CONN_6, symbol CONN_6
Connections:
- wire segments 33 -> 35
Other:
- moved on the sheet: K2
Changed lines of the file:
@@
-EESchema Schematic File Version 2  date Mon 01 Jun 2015 18:53:27 BST
+EESchema Schematic File Version 2  date Sun 05 Jul 2015 19:04:22 BST
 LIBS:quantracker
 LIBS:stm32
@@
 $Descr A4 11700 8267
 encoding utf-8
-Sheet 4 4
+Sheet 5 5
 Title ""
-Date "1 jun 2015"
+Date "5 jul 2015"
 Rev ""
 Comp ""
@@
 Comment4 ""
 $EndDescr
+$Comp
+L CONN_3 K2
+U 1 1 55520FE6
+P 2500 6200
+F 0 "K2" V 2450 6200 50  0000 C CNN
+F 1 "CONN_3" V 2550 6200 40  0000 C CNN
+	1    2500 6200
+	-1   0    0    -1
+$EndComp
+Wire Wire Line
+	6950 3050 6700 3050
+Wire Wire Line
+	4450 3650 4750 3650
+Wire Wire Line
+	8400 1250 8600 1250
+Wire Wire Line
+	7850 1000 7650 1000
+Wire Wire Line
+	8600 1000 8350 1000
+Wire Wire Line
+	7050 3950 6700 3950
+Wire Wire Line
+	7000 3850 6700 3850
+Wire Wire Line
+	7000 4050 6700 4050
+Wire Wire Line
+	5850 4900 5850 4750
+Wire Wire Line
+	5550 4900 5550 4750
+Wire Wire Line
+	7000 3650 6700 3650
+Wire Wire Line
+	7000 3350 6700 3350
+Wire Wire Line
+	4750 4250 4500 4250
+Wire Wire Line
+	4750 3450 4350 3450
+Wire Wire Line
+	4750 2950 4450 2950
+Wire Wire Line
+	6850 2750 6700 2750
+Wire Wire Line
+	4750 3050 4450 3050
+Wire Wire Line
+	4750 3150 4450 3150
+Wire Wire Line
+	4750 3350 4300 3350
+Wire Wire Line
+	4750 4150 4500 4150
+Wire Wire Line
+	7000 3250 6700 3250
+Wire Wire Line
+	7000 3450 6700 3450
+Wire Wire Line
+	7000 3750 6700 3750
+Wire Wire Line
+	5750 4900 5750 4750
+Wire Wire Line
+	5950 4900 5950 4750
+Wire Wire Line
+	4750 4050 4450 4050
+Wire Wire Line
+	7000 4250 6700 4250
+Wire Wire Line
+	4750 2850 4450 2850
+Wire Wire Line
+	6850 2650 6700 2650
+Wire Wire Line
+	7900 1250 7650 1250
+Wire Wire Line
+	4750 3550 4450 3550
+Wire Wire Line
+	6950 2950 6700 2950
 Wire Wire Line
 	4750 2550 4400 2550
 Wire Wire Line
-	6950 2950 6700 2950
-Wire Wire Line
-	4750 3550 4450 3550
-Wire Wire Line
-	7900 1250 7650 1250
-Wire Wire Line
-	6850 2650 6700 2650
-Wire Wire Line
-	4750 2850 4450 2850
-Wire Wire Line
-	7000 4250 6700 4250
-Wire Wire Line
-	4750 4050 4450 4050
-Wire Wire Line
-	5950 4900 5950 4750
-Wire Wire Line
-	5750 4900 5750 4750
-Wire Wire Line
-	7000 3750 6700 3750
-Wire Wire Line
-	7000 3450 6700 3450
-Wire Wire Line
-	7000 3250 6700 3250
-Wire Wire Line
-	4750 4150 4500 4150
-Wire Wire Line
-	4750 3350 4300 3350
-Wire Wire Line
-	4750 3150 4450 3150
-Wire Wire Line
-	4750 3050 4450 3050
-Wire Wire Line
-	6850 2750 6700 2750
-Wire Wire Line
-	4750 2950 4450 2950
-Wire Wire Line
-	4750 3450 4350 3450
-Wire Wire Line
-	4750 4250 4500 4250
-Wire Wire Line
-	7000 3350 6700 3350
-Wire Wire Line
-	7000 3650 6700 3650
-Wire Wire Line
-	5550 4900 5550 4750
-Wire Wire Line
-	5850 4900 5850 4750
-Wire Wire Line
-	7000 4050 6700 4050
-Wire Wire Line
-	7000 3850 6700 3850
-Wire Wire Line
-	7050 3950 6700 3950
-Wire Wire Line
-	8600 1000 8350 1000
-Wire Wire Line
-	7850 1000 7650 1000
-Wire Wire Line
-	8400 1250 8600 1250
-Wire Wire Line
-	4450 3650 4750 3650
-Wire Wire Line
-	6950 3050 6700 3050
+	8400 4700 8400 4650
+Wire Wire Line
+	2600 4400 2650 4400
+Text HLabel 2650 4400 2    60   Output ~ 0
+3.3VO
 Text HLabel 4400 2550 0    60   Input ~ 0
 MCU_GND
@@
 	0    1    1    0
 $EndComp
-Text Notes 1950 5050 2    60   ~ 0
+Text Notes 1750 4350 2    60   ~ 0
 Video Out
-Text Notes 2000 4600 2    60   ~ 0
+Text Notes 1700 4100 2    60   ~ 0
 Video In
-$Comp
-L CONN_3 K2
-U 1 1 55520FE6
-P 1850 6150
-F 0 "K2" V 1800 6150 50  0000 C CNN
-F 1 "CONN_3" V 1900 6150 40  0000 C CNN
-	1    1850 6150
-	-1   0    0    -1
-$EndComp
 Text Notes 1700 2250 2    60   ~ 0
 GPS
@@
 Text Notes 2050 1250 2    60   ~ 0
 Magnetometer
-$Comp
-L CONN_6 P4
-U 1 1 55520DE1
-P 1850 1650
-F 0 "P4" V 1800 1650 60  0000 C CNN
-F 1 "CONN_6" V 1900 1650 60  0000 C CNN
-	1    1850 1650
-	-1   0    0    1
-$EndComp
 Text HLabel 4450 2850 0    60   Output ~ 0
 5VOut
@@
 Text HLabel 7000 4250 2    60   Output ~ 0
 LED2
-Text HLabel 7000 3850 2    60   Output ~ 0
+Text HLabel 7000 3850 2    60   Input ~ 0
 MAG_RDY
 Text HLabel 7000 3650 2    60   Output ~ 0

Commit message: ground tracker schematic mods
Connections:
- net labels added: EXTI1, FRAM_NCS, SPI_NCS
- net labels removed: LED1, MAG_RDY
Other:
- note added: "or QDRT"
Changed lines of the file:
@@
-EESchema Schematic File Version 2  date Sun 05 Jul 2015 19:04:22 BST
+EESchema Schematic File Version 2  date Thu 10 Dec 2015 12:44:52 GMT
 LIBS:quantracker
 LIBS:stm32
@@
 Sheet 5 5
 Title ""
-Date "5 jul 2015"
+Date "10 dec 2015"
 Rev ""
 Comp ""
@@
 Comment4 ""
 $EndDescr
+Text Notes 1200 3550 0    60   ~ 0
+or QDRT
+Text HLabel 4450 3050 0    60   Input ~ 0
+EXTI1
+Text HLabel 4450 2950 0    60   Output ~ 0
+FRAM_NCS
 $Comp
 L CONN_3 K2
@@
 Text HLabel 7000 4250 2    60   Output ~ 0
 LED2
-Text HLabel 7000 3850 2    60   Input ~ 0
-MAG_RDY
+Text HLabel 7000 3850 2    60   Output ~ 0
+SPI_NCS
 Text HLabel 7000 3650 2    60   Output ~ 0
 LCD_TXO
-Text HLabel 4450 2950 0    60   Input ~ 0
+Text HLabel 4500 3850 0    60   Input ~ 0
 BATT_LEVEL_IN
 Text HLabel 7000 3750 2    60   Output ~ 0
@@
 Text HLabel 4450 3650 0    60   Input ~ 0
 USART4_TXO
-Text HLabel 4450 3150 0    60   Output ~ 0
-LED1
-Text HLabel 4450 3050 0    60   Output ~ 0
+Text HLabel 4500 3950 0    60   Output ~ 0
 PAN_MOTOR_DIR
 $Comp

Commit message: old mods updated
Parts:
- M1: value OSD_V2_1 -> OSD_V2_2; symbol OSD_V2_1 -> OSD_v2_1
- R17, R18: symbol R -> R-RESCUE-tracker_using_quantracker_osd
Connections:
- net labels added: PUSH_BUTTON
Other:
- note added: "QDRT"
- note removed: "PUSH_BUTTON"
Changed lines of the file:
@@
-EESchema Schematic File Version 2  date Thu 10 Dec 2015 12:44:52 GMT
+EESchema Schematic File Version 2
+LIBS:tracker_using_quantracker_osd-rescue
 LIBS:quantracker
 LIBS:stm32
@@
 LIBS:memory
 LIBS:xilinx
-LIBS:special
 LIBS:microcontrollers
 LIBS:dsp
@@
 LIBS:mc34931
 LIBS:tracker_using_quantracker_osd-cache
-EELAYER 25  0
+EELAYER 25 0
 EELAYER END
-$Descr A4 11700 8267
+$Descr A4 11693 8268
 encoding utf-8
 Sheet 5 5
@@
 F 0 "K2" V 2450 6200 50  0000 C CNN
 F 1 "CONN_3" V 2550 6200 40  0000 C CNN
+F 2 "" H 2500 6200 60  0001 C CNN
+F 3 "" H 2500 6200 60  0001 C CNN
 	1    2500 6200
 	-1   0    0    -1
@@
 Text HLabel 6950 2950 2    60   Input ~ 0
 LCD_SDA
-Text Notes 7450 4100 0    60   ~ 0
-PUSH_BUTTON
 Text Notes 7950 3000 0    60   ~ 0
 I2C1_SDA/TIM4_CH2\n
@@
 PAN_SERVO_PWM
 $Comp
-L R R18
+L R-RESCUE-tracker_using_quantracker_osd R18
 U 1 1 55521193
 P 8150 1250
 F 0 "R18" V 8230 1250 50  0000 C CNN
 F 1 "R" V 8150 1250 50  0000 C CNN
+F 2 "" H 8150 1250 60  0001 C CNN
+F 3 "" H 8150 1250 60  0001 C CNN
 	1    8150 1250
 	0    1    1    0
@@
 TILT_SERVO_PWM_RAW
 $Comp
-L R R17
+L R-RESCUE-tracker_using_quantracker_osd R17
 U 1 1 555210EC
 P 8100 1000
 F 0 "R17" V 8180 1000 50  0000 C CNN
 F 1 "R" V 8100 1000 50  0000 C CNN
+F 2 "" H 8100 1000 60  0001 C CNN
+F 3 "" H 8100 1000 60  0001 C CNN
 	1    8100 1000
 	0    1    1    0
@@
 F 0 "P5" V 1800 2550 50  0000 C CNN
 F 1 "CONN_4" V 1900 2550 50  0000 C CNN
+F 2 "" H 1850 2550 60  0001 C CNN
+F 3 "" H 1850 2550 60  0001 C CNN
 	1    1850 2550
 	-1   0    0    1
@@
 PAN_MOTOR_DIR
 $Comp
-L OSD_V2_1 M1
+L OSD_v2_1 M1
 U 1 1 5551CEC6
 P 5700 3350
 F 0 "M1" H 5750 3100 60  0000 C CNN
-F 1 "OSD_V2_1" H 5700 3350 60  0000 C CNN
+F 1 "OSD_V2_2" H 5700 3350 60  0000 C CNN
+F 2 "" H 5700 3350 60  0001 C CNN
+F 3 "" H 5700 3350 60  0001 C CNN
 	1    5700 3350
 	1    0    0    -1
 $EndComp
+Text Notes 7575 3000 0    60   ~ 0
+QDRT
+Text HLabel 4450 3150 0    60   Input ~ 0
+PUSH_BUTTON
 $EndSCHEMATC
