File: ground/tracker/v2/hardware/pan_motor.sch (KiCad schematic (older format))
At the start: 16 parts

Commit message: pan_motor servo initla draft aded, not tested yet
Parts:
- removed R? (x4): R, symbol R
- removed U?: 74HC04, symbol 74HC04
- added C? (x2): C, symbol C
- added Q?: MOS_N, symbol MOS_N
- added R?: 27.4K, symbol R
- added R? (x5): 100R, symbol R
- added R?: 1.7K, symbol R
- added R?: 3.3K, symbol R
- added R? (x2): 10K, symbol R
- added R?: 4K7, symbol R
- added U?: LM6132, symbol LM358
- R? (x2): value R -> 100K
- R? (x3): value R -> 27.4K
- U? (x2): value LM358 -> LM6132
Connections:
- net labels added: +12V, ENCODERB, ENCODER_A, PAN_MOTOR_5V, PAN_MOTOR_CURRENT, PAN_MOTOR_EMF, PAN_MOTOR_GND, PAN_MOTOR_PWM
- net labels removed: 5VO, AZIMUTH_MOTOR_CURRENT, AZIMUTH_MOTOR_DIR, AZIMUTH_MOTOR_GND, AZIMUTH_MOTOR_PWM, AZIMUTH_MOTOR_SPEED, ENC5V, ENCA, ENCB, ENCGND, GND, NOT_AZIMUTH_MOTOR_DIR
- wire segments 38 -> 85
Other:
- note added: "using ACS712 hall effect current sensor"
- note removed: "2V"
- moved on the sheet: K?, R?, U?A

Commit message: update ground V2 schematic
Parts:
- removed P?: CONN_2, symbol CONN_2
- removed P?: CONN_4, symbol CONN_4
- added D?: DIODESCH, symbol DIODESCH
- added P?: CONN_5, symbol CONN_5
- added R? (x2): 330R, symbol R
- C1, C2: renamed from C?; value C -> 0.1uF
- R11: renamed from R?; value 1.7K -> 17K
- R12: renamed from R?; value 3.3K -> 33K
- gave numbers to parts that had none: 18
Connections:
- wire segments 85 -> 89

Commit message: velocity pan servo working though sometimes sticks for some reason, maybe after invalid text comand input
Parts:
- added C?: 20nF, symbol C
- added C? (x2): 10nF, symbol C
Connections:
- wire segments 89 -> 81
Other:
- moved on the sheet: R7
Changed lines of the file:
@@
-EESchema Schematic File Version 2  date Thu 21 May 2015 21:44:38 BST
+EESchema Schematic File Version 2  date Thu 28 May 2015 15:49:42 BST
 LIBS:quantracker
 LIBS:stm32
@@
 Sheet 2 3
 Title ""
-Date "21 may 2015"
+Date "28 may 2015"
 Rev ""
 Comp ""
@@
 Comment4 ""
 $EndDescr
+Connection ~ 5350 2400
+Wire Wire Line
+	5650 2300 5650 2400
+Wire Wire Line
+	5650 2400 5350 2400
+Connection ~ 5350 1650
+Connection ~ 5650 1650
+Wire Wire Line
+	5350 1650 5650 1650
+Connection ~ 3800 3350
+Wire Wire Line
+	3800 3150 3800 3650
+Wire Wire Line
+	3800 3650 3950 3650
+Wire Wire Line
+	9000 6300 8650 6300
+Wire Wire Line
+	8650 6300 8650 6100
+Wire Wire Line
+	8650 6100 8400 6100
+Connection ~ 1800 6500
+Wire Wire Line
+	1800 6500 1800 5850
+Wire Wire Line
+	3450 4900 3450 4700
+Wire Wire Line
+	3450 4700 1600 4700
+Wire Wire Line
+	3450 5950 3450 6500
+Wire Wire Line
+	3450 6500 1650 6500
+Wire Wire Line
+	5350 7200 5350 7400
+Wire Wire Line
+	5350 7400 5250 7400
+Connection ~ 2450 2250
+Wire Wire Line
+	2450 1800 2450 2250
+Wire Wire Line
+	1800 2100 1800 2250
+Wire Wire Line
+	1800 2250 2600 2250
+Wire Wire Line
+	5400 2500 5350 2500
+Wire Wire Line
+	5350 2500 5350 2250
+Wire Wire Line
+	7350 3850 7350 3750
+Wire Wire Line
+	8900 3850 8450 3850
+Wire Wire Line
+	8000 6100 7650 6100
+Connection ~ 4500 3150
+Wire Wire Line
+	4500 3350 4400 3350
+Wire Wire Line
+	6950 3150 6450 3150
+Wire Wire Line
+	8900 3150 7450 3150
+Wire Wire Line
+	8900 2950 8650 2950
+Wire Wire Line
+	7850 6600 5200 6600
+Wire Wire Line
+	9000 6600 8350 6600
+Wire Wire Line
+	7100 6400 6750 6400
+Wire Wire Line
+	9000 6400 7600 6400
+Wire Wire Line
+	2850 5750 3150 5750
+Wire Wire Line
+	5350 950  5350 1050
+Wire Wire Line
+	2600 2750 2250 2750
+Wire Wire Line
+	3500 2750 3100 2750
+Wire Wire Line
+	4800 2850 4500 2850
+Wire Wire Line
+	5300 2650 5950 2650
+Wire Wire Line
+	8900 2750 5950 2750
+Wire Wire Line
+	5950 2750 5950 2650
+Wire Wire Line
+	8900 2850 5300 2850
+Wire Wire Line
+	4800 2650 4500 2650
+Wire Wire Line
+	4400 3150 4600 3150
+Wire Wire Line
+	4600 3150 4600 2850
+Connection ~ 4600 2850
+Wire Wire Line
+	3900 3150 3350 3150
+Wire Wire Line
+	3350 3150 3350 2750
+Connection ~ 3350 2750
+Wire Wire Line
+	5350 1750 5350 1550
+Wire Wire Line
+	4600 2650 4600 1700
+Wire Wire Line
+	4600 1700 5350 1700
+Connection ~ 5350 1700
+Connection ~ 4600 2650
+Connection ~ 5950 4550
+Wire Wire Line
+	5950 4550 5950 4950
+Wire Wire Line
+	5950 4950 7150 4950
+Wire Wire Line
+	7150 4950 7150 4650
+Wire Wire Line
+	7350 3750 8900 3750
+Wire Wire Line
+	7150 4650 7100 4650
+Wire Wire Line
+	4500 4550 5050 4550
+Wire Wire Line
+	5550 4550 6100 4550
+Wire Wire Line
+	3700 5500 3450 5500
+Wire Wire Line
+	6750 6500 7450 6500
+Wire Wire Line
+	7950 6500 9000 6500
+Wire Wire Line
+	6750 6700 9000 6700
+Wire Wire Line
+	8650 3050 8900 3050
+Wire Wire Line
+	7900 3250 8900 3250
+Wire Wire Line
+	6450 3250 7400 3250
+Wire Wire Line
+	3900 3350 3800 3350
+Connection ~ 3800 3150
+Wire Wire Line
+	8900 3950 8450 3950
+Wire Wire Line
+	7350 4550 7350 4350
+Wire Wire Line
+	7100 4450 7350 4450
+Connection ~ 7350 4450
+Wire Wire Line
+	1800 1200 1800 900
+Wire Wire Line
+	1700 900  2450 900
+Wire Wire Line
+	2450 900  2450 1400
+Connection ~ 1800 900
+Wire Wire Line
+	5350 6700 5350 6600
+Connection ~ 5350 6600
+Wire Wire Line
+	3450 5550 3450 5400
+Wire Wire Line
+	3000 5850 3000 5750
+Connection ~ 3000 5750
+Wire Wire Line
+	3000 6500 3000 6350
+Connection ~ 3000 6500
+Wire Wire Line
+	1800 5450 1800 4700
+Connection ~ 1800 4700
+Wire Wire Line
+	7200 5250 7350 5250
+Wire Wire Line
+	7350 5250 7350 5050
+Wire Wire Line
+	4350 3650 4500 3650
+Wire Wire Line
+	4500 3650 4500 3150
+Connection ~ 4500 3350
+Wire Wire Line
+	5650 1900 5650 1500
+Wire Wire Line
+	5250 950  5650 950
+Wire Wire Line
+	5650 950  5650 1100
+Connection ~ 5350 950
+$Comp
+L C C?
+U 1 1 55672A56
+P 5650 1300
+F 0 "C?" H 5700 1400 50  0000 L CNN
+F 1 "10nF" H 5700 1200 50  0000 L CNN
+	1    5650 1300
+	1    0    0    -1
+$EndComp
+$Comp
+L C C?
+U 1 1 55672A53
+P 5650 2100
+F 0 "C?" H 5700 2200 50  0000 L CNN
+F 1 "10nF" H 5700 2000 50  0000 L CNN
+	1    5650 2100
+	1    0    0    -1
+$EndComp
+$Comp
+L C C?
+U 1 1 55672A20
+P 4150 3650
+F 0 "C?" H 4200 3750 50  0000 L CNN
+F 1 "20nF" H 4200 3550 50  0000 L CNN
+	1    4150 3650
+	0    1    1    0
+$EndComp
 $Comp
 L R R?
@@
 	0    1    1    0
 $EndComp
-Wire Wire Line
-	9000 6300 8650 6300
-Wire Wire Line
-	8650 6300 8650 6100
-Wire Wire Line
-	8650 6100 8400 6100
-Connection ~ 1800 6500
-Wire Wire Line
-	1800 6500 1800 5850
-Wire Wire Line
-	3450 4900 3450 4700
-Wire Wire Line
-	3450 4700 1800 4700
-Wire Wire Line
-	1800 4700 1600 4700
-Wire Wire Line
-	3450 5950 3450 6500
-Wire Wire Line
-	3450 6500 3000 6500
-Wire Wire Line
-	3000 6500 1800 6500
-Wire Wire Line
-	1800 6500 1650 6500
-Wire Wire Line
-	5350 7200 5350 7400
-Wire Wire Line
-	5350 7400 5250 7400
-Connection ~ 2450 2250
-Wire Wire Line
-	2450 1800 2450 2250
-Wire Wire Line
-	1800 2100 1800 2250
-Wire Wire Line
-	1800 2250 2450 2250
-Wire Wire Line
-	2450 2250 2600 2250
-Wire Wire Line
-	5400 2500 5350 2500
-Wire Wire Line
-	5350 2500 5350 2250
-Wire Wire Line
-	7350 3850 7350 3750
-Wire Wire Line
-	8900 3850 8450 3850
-Wire Wire Line
-	8000 6100 7650 6100
-Connection ~ 4500 3150
-Wire Wire Line
-	4500 3150 4500 3350
-Wire Wire Line
-	4500 3350 4400 3350
-Wire Wire Line
-	6950 3150 6450 3150
-Wire Wire Line
-	8900 3150 7450 3150
-Wire Wire Line
-	8900 2950 8650 2950
-Wire Wire Line
-	7850 6600 5350 6600
-Wire Wire Line
-	5350 6600 5200 6600
-Wire Wire Line
-	9000 6600 8350 6600
-Wire Wire Line
-	7100 6400 6750 6400
-Wire Wire Line
-	9000 6400 7600 6400
-Wire Wire Line
-	2850 5750 3000 5750
-Wire Wire Line
-	3000 5750 3150 5750
-Wire Wire Line
-	5350 1150 5350 1050
-Wire Wire Line
-	5350 1050 5250 1050
-Wire Wire Line
-	3500 2750 3350 2750
-Wire Wire Line
-	2600 2750 2250 2750
-Wire Wire Line
-	3350 2750 3100 2750
-Wire Wire Line
-	4800 2850 4600 2850
-Wire Wire Line
-	4600 2850 4500 2850
-Wire Wire Line
-	5300 2650 5950 2650
-Wire Wire Line
-	8900 2750 5950 2750
-Wire Wire Line
-	5950 2750 5950 2650
-Wire Wire Line
-	8900 2850 5300 2850
-Wire Wire Line
-	4800 2650 4600 2650
-Wire Wire Line
-	4600 2650 4500 2650
-Wire Wire Line
-	4400 3150 4500 3150
-Wire Wire Line
-	4500 3150 4600 3150
-Wire Wire Line
-	4600 3150 4600 2850
-Connection ~ 4600 2850
-Wire Wire Line
-	3900 3150 3800 3150
-Wire Wire Line
-	3800 3150 3350 3150
-Wire Wire Line
-	3350 3150 3350 2750
-Connection ~ 3350 2750
-Wire Wire Line
-	5350 1750 5350 1700
-Wire Wire Line
-	5350 1700 5350 1650
-Wire Wire Line
-	4600 2650 4600 1700
-Wire Wire Line
-	4600 1700 5350 1700
-Connection ~ 5350 1700
-Connection ~ 4600 2650
-Connection ~ 5950 4550
-Wire Wire Line
-	5950 4550 5950 4950
-Wire Wire Line
-	5950 4950 7150 4950
-Wire Wire Line
-	7150 4950 7150 4650
-Wire Wire Line
-	7350 3750 8900 3750
-Wire Wire Line
-	7150 4650 7100 4650
-Wire Wire Line
-	5550 4550 5950 4550
-Wire Wire Line
-	4500 4550 5050 4550
-Wire Wire Line
-	5950 4550 6100 4550
-Wire Wire Line
-	3700 5500 3450 5500
-Wire Wire Line
-	6750 6500 7450 6500
-Wire Wire Line
-	7950 6500 9000 6500
-Wire Wire Line
-	6750 6700 9000 6700
-Wire Wire Line
-	8650 3050 8900 3050
-Wire Wire Line
-	7900 3250 8900 3250
-Wire Wire Line
-	6450 3250 7400 3250
-Wire Wire Line
-	3900 3350 3800 3350
-Wire Wire Line
-	3800 3350 3800 3150
-Connection ~ 3800 3150
-Wire Wire Line
-	8900 3950 8450 3950
-Wire Wire Line
-	7350 4550 7350 4450
-Wire Wire Line
-	7350 4450 7350 4350
-Wire Wire Line
-	7100 4450 7350 4450
-Connection ~ 7350 4450
-Wire Wire Line
-	1800 1200 1800 900
-Wire Wire Line
-	1700 900  1800 900
-Wire Wire Line
-	1800 900  2450 900
-Wire Wire Line
-	2450 900  2450 1400
-Connection ~ 1800 900
-Wire Wire Line
-	5350 6700 5350 6600
-Connection ~ 5350 6600
-Wire Wire Line
-	3450 5550 3450 5400
-Wire Wire Line
-	3000 5850 3000 5750
-Connection ~ 3000 5750
-Wire Wire Line
-	3000 6500 3000 6350
-Connection ~ 3000 6500
-Wire Wire Line
-	1800 5450 1800 4700
-Connection ~ 1800 4700
-Wire Wire Line
-	7200 5250 7350 5250
-Wire Wire Line
-	7350 5250 7350 5050
 $Comp
 L R R?
@@
 Text HLabel 2250 2750 0    60   Output ~ 0
 PAN_MOTOR_EMF
-Text HLabel 5250 1050 0    60   Input ~ 0
+Text HLabel 5250 950  0    60   Input ~ 0
 3.3VO
 $Comp
@@
 L R R7
 U 1 1 55534465
-P 5350 1400
-F 0 "R7" V 5430 1400 50  0000 C CNN
-F 1 "27.4K" V 5350 1400 50  0000 C CNN
-	1    5350 1400
-	1    0    0    -1
-$EndComp
+P 5350 1300
+F 0 "R7" V 5430 1300 50  0000 C CNN
+F 1 "27.4K" V 5350 1300 50  0000 C CNN
+	1    5350 1300
+	1    0    0    -1
+$EndComp
