File: ground/tracker/v2/hardware/pan_motor.sch (KiCad schematic (older format))
At the start: 29 parts, among them K1 CONN_3, P1 CONN_6, Q1 MOS_N, U1 LM6132

Commit message: added FreeCAD design files for V2 tracker
Parts:
- removed D?: DIODESCH, symbol DIODESCH
- removed K1: CONN_3, symbol CONN_3
- removed P1: CONN_6, symbol CONN_6
- removed P?: CONN_5, symbol CONN_5
- removed R10, R14: 100R, symbol R
- added C?: 33nF, symbol C
- added C?: C, symbol C
- added K?: CONN_3, symbol CONN_3
- added R?: 220R, symbol R
- added R?: R, symbol R
- added U?: MC34931, symbol MC34931
Connections:
- net labels removed: ENCODERB, ENCODER_A, NOT_PAN_MOTOR_DIR, PAN_MOTOR_5V, RAW_CURRENT_IN
- wire segments 81 -> 131
Other:
- note removed: "PanMotor Ctrl"
- note removed: "PanMotorCurrent"
- note removed: "using ACS712 hall effect current sensor"
- moved on the sheet: C1, Q1, R1, R11, R12, R13, R15, R16, R2, R9, R?, U1B

Commit message: old mods updated
Parts:
- C1, C2, C? (x5): symbol C -> C-RESCUE-tracker_using_quantracker_osd
- R1, R11, R12, R13, R15, R16, R2, R3, R4, R5, R6, R7, R8, R9, R? (x4): symbol R -> R-RESCUE-tracker_using_quantracker_osd
Connections:
- net at R?.1, U1.5 (+), U?.3 (FB): no longer C?.1

Commit message: tracker v2 commit bundle
Changed lines of the file:
@@
 $Descr A4 11693 8268
 encoding utf-8
-Sheet 4 5
+Sheet 4 6
 Title ""
 Date "10 dec 2015"
@@
 	10000 4700 9800 4700
 Wire Wire Line
-	9800 5600 9800 4700
+	9800 4700 9800 5600
 Wire Wire Line
-	6400 5600 9800 5600
+	9800 5600 6400 5600
 Connection ~ 9450 4600
 Wire Wire Line
