File: ground/tracker/v2/hardware/magnetometer.sch (KiCad schematic (older format))
At the start: 7 parts

Commit message: old mods updated
Parts:
- 100R?, R? (x5): symbol R -> R-RESCUE-tracker_using_quantracker_osd
Connections:
- wire segments 25 -> 22
Changed lines of the file:
@@
-EESchema Schematic File Version 2  date Thu 10 Dec 2015 12:44:52 GMT
+EESchema Schematic File Version 2
+LIBS:tracker_using_quantracker_osd-rescue
 LIBS:quantracker
 LIBS:stm32
@@
 LIBS:memory
 LIBS:xilinx
-LIBS:special
 LIBS:microcontrollers
 LIBS:dsp
@@
 LIBS:mc34931
 LIBS:tracker_using_quantracker_osd-cache
-EELAYER 25  0
+EELAYER 25 0
 EELAYER END
-$Descr A4 11700 8267
+$Descr A4 11693 8268
 encoding utf-8
 Sheet 2 5
@@
 MAG_SCL
 $Comp
-L R R?
+L R-RESCUE-tracker_using_quantracker_osd R?
 U 1 1 55996006
 P 5750 4000
 F 0 "R?" V 5830 4000 50  0000 C CNN
 F 1 "100R" V 5750 4000 50  0000 C CNN
+F 2 "" H 5750 4000 60  0001 C CNN
+F 3 "" H 5750 4000 60  0001 C CNN
 	1    5750 4000
 	0    1    1    0
 $EndComp
 $Comp
-L R 100R?
+L R-RESCUE-tracker_using_quantracker_osd 100R?
 U 1 1 55996005
 P 5250 3100
 F 0 "100R?" V 5330 3100 50  0000 C CNN
 F 1 "R" V 5300 3300 50  0000 C CNN
+F 2 "" H 5250 3100 60  0001 C CNN
+F 3 "" H 5250 3100 60  0001 C CNN
 	1    5250 3100
 	0    1    1    0
 $EndComp
 $Comp
-L R R?
+L R-RESCUE-tracker_using_quantracker_osd R?
 U 1 1 55996004
 P 4350 2750
 F 0 "R?" V 4450 2850 50  0000 C CNN
 F 1 "100R" V 4350 2750 50  0000 C CNN
+F 2 "" H 4350 2750 60  0001 C CNN
+F 3 "" H 4350 2750 60  0001 C CNN
 	1    4350 2750
 	0    1    1    0
 $EndComp
 $Comp
-L R R?
+L R-RESCUE-tracker_using_quantracker_osd R?
 U 1 1 55996003
 P 5300 3650
 F 0 "R?" V 5380 3650 50  0000 C CNN
 F 1 "10K" V 5300 3650 50  0000 C CNN
+F 2 "" H 5300 3650 60  0001 C CNN
+F 3 "" H 5300 3650 60  0001 C CNN
 	1    5300 3650
 	1    0    0    -1
@@
 3.3VO
 $Comp
-L R R?
+L R-RESCUE-tracker_using_quantracker_osd R?
 U 1 1 55996002
 P 5550 2800
 F 0 "R?" V 5630 2800 50  0000 C CNN
 F 1 "10K" V 5550 2800 50  0000 C CNN
+F 2 "" H 5550 2800 60  0001 C CNN
+F 3 "" H 5550 2800 60  0001 C CNN
 	1    5550 2800
 	1    0    0    -1
 $EndComp
 $Comp
-L R R?
+L R-RESCUE-tracker_using_quantracker_osd R?
 U 1 1 55996001
 P 4650 2450
 F 0 "R?" V 4730 2450 50  0000 C CNN
 F 1 "10K" V 4650 2450 50  0000 C CNN
+F 2 "" H 4650 2450 60  0001 C CNN
+F 3 "" H 4650 2450 60  0001 C CNN
 	1    4650 2450
 	1    0    0    -1
@@
 	3550 2900 4650 2900
 Wire Wire Line
-	4650 2750 4750 2750
-Wire Wire Line
-	4600 2750 4650 2750
+	4600 2750 4750 2750
 Connection ~ 5550 3100
 Wire Wire Line
@@
 	4450 4000 4450 3100
 Wire Wire Line
-	5300 4000 4450 4000
-Wire Wire Line
-	5500 4000 5300 4000
+	4450 4000 5500 4000
 Wire Wire Line
 	6000 4000 6150 4000
 Wire Wire Line
-	5550 3100 5500 3100
-Wire Wire Line
-	5600 3100 5550 3100
+	5500 3100 5600 3100
 Wire Wire Line
 	4650 2700 4650 2750
@@
 F 0 "P?" V 3100 3000 50  0000 C CNN
 F 1 "CONN_5" V 3200 3000 50  0000 C CNN
+F 2 "" H 3150 3000 60  0001 C CNN
+F 3 "" H 3150 3000 60  0001 C CNN
 	1    3150 3000
 	-1   0    0    1
