File: air/osd/hardware/64_pin_lite/air_osd_v2_2/kicad_project/mcu.sch (KiCad schematic (older format))
At the start: 29 parts, among them P1 SIL2, P6 Pad, P7 Pad, P8 Pad, U1 SI501, U2 STM32F405RGT6, U3 74LVC1G86

Commit message: changed diode pins side to comply with IPC-7351 2005 (dont have later spec)
Parts:
- D1: value Red Led -> Red_Led
Changed lines of the file:
@@
-EESchema Schematic File Version 2  date Sun 21 Jun 2015 14:24:06 BST
+EESchema Schematic File Version 2  date Thu 25 Jun 2015 08:05:44 BST
+LIBS:conn_20
+LIBS:conn_6
+LIBS:conn_5
+LIBS:conn_3
+LIBS:conn_2
 LIBS:power
 LIBS:device
@@
 LIBS:contrib
 LIBS:valves
+LIBS:diodesch_ipc7531_2005
 LIBS:osd-cache
 EELAYER 25  0
@@
 Sheet 2 8
 Title ""
-Date "20 jun 2015"
+Date "25 jun 2015"
 Rev ""
 Comp ""
@@
 P 6650 1775
 F 0 "D1" H 6650 1875 50  0000 C CNN
-F 1 "Red Led" V 6400 1475 50  0000 C CNN
+F 1 "Red_Led" V 6400 1475 50  0000 C CNN
 F 2 "0603" H 6650 1775 60  0001 C CNN
 F 3 "D" H 6650 1775 60  0001 C CNN

Commit message: v2.2 pcb hopefully ready to go
Parts:
- removed D1: Red_Led, 0603, symbol LED
- added D1: Red_Led, 0603, symbol LED_IPC-7351_2005
Connections:
- net MCU_GND: now also D1.1 (Ca)
- net RED_LED_RES: now also D1.2 (An)
