File: air/osd/hardware/64_pin_lite/air_osd_v2_2/kicad_project/psu.sch (KiCad schematic (older format))
At the start: 24 parts, among them U4 BD9G101G, U5 LD39015MXXR

Commit message: added Fiducials and settings to get pos file
Parts:
- C12, C40, C42: MFG Name Samsung -> M; MFG Part Num CL10B104KB8SFNC -> P
- C13, C41: MFG Name Taiyo Yuden -> M; MFG Part Num UMK316ABJ475KD-T -> P
- C14: MFG Name Samsung -> M; MFG Part Num CL10B153KB8NNNC -> P
- C15: MFG Name Kemet -> M; MFG Part Num C0603C154K5RACTU -> P
- C16, C17: MFG Name Murata -> M; MFG Part Num GRM31CR61H106KA12L -> P
- C19: MFG Name Samsung -> M; MFG Part Num CL21F106ZPFNNNE -> P
Changed lines of the file:
@@
-EESchema Schematic File Version 2  date Thu 18 Jun 2015 19:52:51 BST
+EESchema Schematic File Version 2  date Fri 19 Jun 2015 22:46:51 BST
 LIBS:lm358
 LIBS:conn_6
@@
 LIBS:R0link
 LIBS:emi_filter
+LIBS:fiducial
+LIBS:osd-cache
 EELAYER 25  0
 EELAYER END
@@
 Sheet 3 8
 Title "noname.sch"
-Date "18 jun 2015"
+Date "19 jun 2015"
 Rev ""
 Comp ""
@@
 	2250 3200 2300 3200
 Wire Wire Line
-	2300 3450 2300 3200
-Wire Wire Line
-	1650 4600 1650 4300
+	2300 3200 2300 3450
+Wire Wire Line
+	1650 4300 1650 4600
 Wire Wire Line
 	900  4300 2250 4300
@@
 	9950 3300 9550 3300
 Wire Wire Line
-	9550 4000 9550 3300
+	9550 3300 9550 4000
 Connection ~ 9950 3400
 Wire Wire Line
 	9950 3400 10600 3400
 Wire Wire Line
-	9950 3000 10700 3000
-Wire Wire Line
-	9950 4000 9950 3000
+	10700 3000 9950 3000
+Wire Wire Line
+	9950 3000 9950 4000
 Connection ~ 3000 3700
 Wire Wire Line
-	2650 3700 2650 3900
+	2650 3900 2650 3700
 Wire Wire Line
 	2650 3700 3300 3700
@@
 Connection ~ 6150 3250
 Wire Wire Line
-	6450 3250 6150 3250
+	6150 3250 6450 3250
 Wire Wire Line
 	6450 3250 6450 3350
@@
 Connection ~ 5150 3200
 Wire Wire Line
-	5050 6450 5050 4600
+	5050 4600 5050 6450
 Wire Wire Line
 	3400 3600 3300 3600
@@
 Connection ~ 9250 6450
 Wire Wire Line
-	10250 6450 5050 6450
+	5050 6450 10250 6450
 Wire Wire Line
 	8850 4600 8850 4400
@@
 	8050 6450 8050 5550
 Wire Wire Line
-	1700 3750 1600 3750
+	1600 3750 1700 3750
 Wire Wire Line
 	1000 3750 800  3750
@@
 F 1 "0.1uF" H 1900 3900 50  0000 L CNN
 F 2 "0603" H 1850 4000 60  0001 C CNN
-F 3 "www.samsungsemi.com/global/support/library/product-catalog/__icsFiles/afieldfile/2014/11/13/MLCC.pdf" H 7900 6325 60  0001 C CNN
-F 4 "Samsung" H 7900 6325 60  0001 C CNN "MFG Name"
-F 5 "CL10B104KB8SFNC" H 7900 6325 60  0001 C CNN "MFG Part Num"
+F 3 "D" H 7900 6325 60  0001 C CNN
+F 4 "M" H 7900 6325 60  0001 C CNN "MFG Name"
+F 5 "P" H 7900 6325 60  0001 C CNN "MFG Part Num"
 F 6 "Capacitor/0.1uF/50V/+-10%/X7R/0603" H 7900 6325 60  0001 C CNN "Description"
 	1    1850 4000
@@
 HUB_+3.3V
 $Comp
-L PWR_FLAG #FLG2
+L PWR_FLAG #FLG01
 U 1 1 54F72D02
 P 7600 3050
-F 0 "#FLG2" H 7600 3320 30  0001 C CNN
+F 0 "#FLG01" H 7600 3320 30  0001 C CNN
 F 1 "PWR_FLAG" H 7600 3280 30  0000 C CNN
 	1    7600 3050
@@
 F 2 "0603" H 2650 4100 60  0001 C CNN
 F 3 "D" H 2650 4100 60  0001 C CNN
-F 4 "Samsung" H 2650 4100 60  0001 C CNN "MFG Name"
-F 5 "CL10B104KB8SFNC" H 2650 4100 60  0001 C CNN "MFG Part Num"
+F 4 "M" H 2650 4100 60  0001 C CNN "MFG Name"
+F 5 "P" H 2650 4100 60  0001 C CNN "MFG Part Num"
 F 6 "Capacitor/0.1uF/50V/X7R/0603" H 2650 4100 60  0001 C CNN "Description"
 	1    2650 4100
@@
 F 2 "1206" H 3000 4100 60  0001 C CNN
 F 3 "D" H 3000 4100 60  0001 C CNN
-F 4 "Taiyo Yuden" H 3000 4100 60  0001 C CNN "MFG Name"
-F 5 "UMK316ABJ475KD-T" H 3000 4100 60  0001 C CNN "MFG Part Num"
+F 4 "M" H 3000 4100 60  0001 C CNN "MFG Name"
+F 5 "P" H 3000 4100 60  0001 C CNN "MFG Part Num"
 F 6 "Capacitor/4.7uF/50V/+-20%/X5R/1206" H 3000 4100 60  0001 C CNN "Description"
 	1    3000 4100
@@
 F 2 "0805" H 9550 4200 60  0001 C CNN
 F 3 "D" H 9550 4200 60  0001 C CNN
-F 4 "Samsung" H 9550 4200 60  0001 C CNN "MFG Name"
-F 5 "CL21F106ZPFNNNE" H 9550 4200 60  0001 C CNN "MFG Part Num"
+F 4 "M" H 9550 4200 60  0001 C CNN "MFG Name"
+F 5 "P" H 9550 4200 60  0001 C CNN "MFG Part Num"
 F 6 "Capacitor/10uF/10V/-20%+80%/Y5V/0805" H 9550 4200 60  0001 C CNN "Description"
 	1    9550 4200
@@
 F 1 "0.15uF" H 6500 3450 50  0000 L CNN
 F 2 "0603" H 6450 3550 60  0001 C CNN
-F 3 "www.kemet.com/Lists/ProductCatalog/Attachments/53/KEM_C1002_X7R_SMD.pdf" H 6450 3550 60  0001 C CNN
-F 4 "Kemet" H 6450 3550 60  0001 C CNN "MFG Name"
-F 5 "C0603C154K5RACTU" H 6450 3550 60  0001 C CNN "MFG Part Num"
+F 3 "D" H 6450 3550 60  0001 C CNN
+F 4 "M" H 6450 3550 60  0001 C CNN "MFG Name"
+F 5 "P" H 6450 3550 60  0001 C CNN "MFG Part Num"
 F 6 "Capacitor/0.15uF/35V/+-10%/X7R/0603" H 6450 3550 60  0001 C CNN "Description"
 	1    6450 3550
@@
 F 2 "1206" H 6750 3950 60  0001 C CNN
 F 3 "D" H 6750 3950 60  0001 C CNN
-F 4 "Murata" H 6750 3950 60  0001 C CNN "MFG Name"
-F 5 "GRM31CR61H106KA12L" H 6750 3950 60  0001 C CNN "MFG Part Num"
+F 4 "M" H 6750 3950 60  0001 C CNN "MFG Name"
+F 5 "P" H 6750 3950 60  0001 C CNN "MFG Part Num"
 F 6 "Capacitor/10uF/50V/+-10%/X5R/1206" H 6750 3950 60  0001 C CNN "Description"
 	1    6750 3950
@@
 200 mA  @ 5V
 $Comp
-L PWR_FLAG #FLG1
+L PWR_FLAG #FLG02
 U 1 1 547116AD
 P 3050 3250
-F 0 "#FLG1" H 3050 3520 30  0001 C CNN
+F 0 "#FLG02" H 3050 3520 30  0001 C CNN
 F 1 "PWR_FLAG" H 3050 3480 30  0000 C CNN
 	1    3050 3250
@@
 F 2 "1206" H 7550 4250 60  0001 C CNN
 F 3 "D" H 7550 4250 60  0001 C CNN
-F 4 "Murata" H 7550 4250 60  0001 C CNN "MFG Name"
-F 5 "GRM31CR61H106KA12L" H 7550 4250 60  0001 C CNN "MFG Part Num"
+F 4 "M" H 7550 4250 60  0001 C CNN "MFG Name"
+F 5 "P" H 7550 4250 60  0001 C CNN "MFG Part Num"
 F 6 "Capacitor/10uF/50V/+-10%/X5R/1206" H 7550 4250 60  0001 C CNN "Description"
 F 7 "10 V" H 7550 4250 60  0001 C CNN "Voltage"
@@
 F 1 "0.1uF" H 2300 3750 50  0000 L CNN
 F 2 "0603" H 2250 3850 60  0001 C CNN
-F 3 "www.samsungsemi.com/global/support/library/product-catalog/__icsFiles/afieldfile/2014/11/13/MLCC.pdf" H 7900 6325 60  0001 C CNN
-F 4 "Samsung" H 7900 6325 60  0001 C CNN "MFG Name"
-F 5 "CL10B104KB8SFNC" H 7900 6325 60  0001 C CNN "MFG Part Num"
+F 3 "D" H 7900 6325 60  0001 C CNN
+F 4 "M" H 7900 6325 60  0001 C CNN "MFG Name"
+F 5 "P" H 7900 6325 60  0001 C CNN "MFG Part Num"
 F 6 "Capacitor/0.1uF/50V/+-10%/X7R/0603" H 7900 6325 60  0001 C CNN "Description"
 	1    2250 3850
@@
 F 2 "0603" H 5150 3500 60  0001 C CNN
 F 3 "D" H 5150 3500 60  0001 C CNN
-F 4 "Samsung" H 5150 3500 60  0001 C CNN "MFG Name"
-F 5 "CL10B153KB8NNNC" H 5150 3500 60  0001 C CNN "MFG Part Num"
+F 4 "M" H 5150 3500 60  0001 C CNN "MFG Name"
+F 5 "P" H 5150 3500 60  0001 C CNN "MFG Part Num"
 F 6 "Capacitor/15nF/50V/+-10%/X7R/0603" H 5150 3500 60  0001 C CNN "Description"
 	1    5150 3500
@@
 F 2 "1206" H 3300 4100 60  0001 C CNN
 F 3 "D" H 3300 4100 60  0001 C CNN
-F 4 "Taiyo Yuden" H 3300 4100 60  0001 C CNN "MFG Name"
-F 5 "UMK316ABJ475KD-T" H 3300 4100 60  0001 C CNN "MFG Part Num"
+F 4 "M" H 3300 4100 60  0001 C CNN "MFG Name"
+F 5 "P" H 3300 4100 60  0001 C CNN "MFG Part Num"
 F 6 "Capacitor/4.7uF/50V/+-20%/X5R/1206" H 3300 4100 60  0001 C CNN "Description"
 	1    3300 4100
