File: air/osd/hardware/64_pin_lite/air_osd_v2_2/kicad_project/psu.sch (KiCad schematic (older format))
At the start: 24 parts, among them U4 BD9G101G, U5 LD39015MXXR

Commit message: changed diode pins side to comply with IPC-7351 2005 (dont have later spec)
Parts:
- removed D6: MBR0530T1G, SOD-123, symbol DIODESCH
- added D6: MBR0530T1G, symbol DIODESCH_IPC7531_2005
- C17: Voltage 10 V -> (none)
- C18: Description Capacitor/0.1uF/10V/+-20%/X7R/0603 -> Capacitor/0.1uF/50V/+-20%/X7R/0603; Voltage 10V -> (none)
- C40: Description Capacitor/0.1uF/50V/X7R/0603 -> Capacitor/0.1uF/50V/+-10%/X7R/0603
- D2: symbol DIODESCH -> DIODESCH_IPC7531_2005; Description Diode/Schottky/30V/500mA/SOD-123 -> Diode/Schottky/30V/0.5A/SOD-123
- D3: value Blue Led -> Blue_Led
- L3: footprint Custom/4mmx4mmx1.8 mm -> LPS4018

Commit message: v2.2 pcb hopefully ready to go
Parts:
- removed D3: Blue_Led, 0603, symbol LED
- added D3: Blue_Led, 0603, symbol LED_IPC-7351_2005
- D2: Description Diode/Schottky/30V/0.5A/SOD-123 -> Diode/Schottky/30V/500mA/SOD-123
- D6: footprint (none) -> SOD-123; Description (none) -> Diode Schottky/30V/500mA/SOD-123; MFG Name (none) -> On Semiconductor; MFG Part Num (none) -> MBR0530T10G
- L2: Description Inductor/22nH/ -> Inductor/22nH/+-10%/0.4R/0603
- L4: Description Inductor/22nH/0603 -> Inductor/22nH/+-10%/0.4R/0603
- L5: Description Bead/EMI supression -> Inductor/Bead/0603
Changed lines of the file:
@@
-EESchema Schematic File Version 2  date Thu 25 Jun 2015 08:05:44 BST
+EESchema Schematic File Version 2  date Thu 25 Jun 2015 13:32:01 BST
 LIBS:conn_20
 LIBS:conn_6
@@
 LIBS:valves
 LIBS:diodesch_ipc7531_2005
+LIBS:led_ipc-7351_2005
 LIBS:osd-cache
 EELAYER 25  0
@@
 Comment4 ""
 $EndDescr
+$Comp
+L LED_IPC-7351_2005 D3
+U 1 1 558BAE9C
+P 7200 3650
+F 0 "D3" H 7200 3500 50  0000 C CNN
+F 1 "Blue_Led" H 7200 3800 50  0000 C CNN
+F 2 "0603" H 7200 3650 60  0001 C CNN
+F 3 "D" H 7200 3650 60  0001 C CNN
+F 4 "M" H 7200 3650 60  0001 C CNN "MFG Name"
+F 5 "P" H 7200 3650 60  0001 C CNN "MFG Part Num"
+F 6 "Led/Blue/0603" H 7200 3650 60  0001 C CNN "Description"
+	1    7200 3650
+	0    -1   -1   0
+$EndComp
 Wire Wire Line
 	2100 3450 2350 3450
@@
 	7950 4600 7950 4350
 Wire Wire Line
-	7200 3850 7200 3950
+	7200 3800 7200 3950
 Connection ~ 7550 4600
 Connection ~ 6150 3250
@@
 Connection ~ 8850 4600
 Wire Wire Line
-	7200 3450 7200 3400
+	7200 3500 7200 3400
 Wire Wire Line
 	7200 3400 7550 3400
@@
 F 0 "D6" H 1950 3550 40  0000 C CNN
 F 1 "MBR0530T1G" H 1950 3350 40  0000 C CNN
+F 2 "SOD-123" H 1950 3450 60  0001 C CNN
+F 3 "D" H 1950 3450 60  0001 C CNN
+F 4 "On Semiconductor" H 1950 3450 60  0001 C CNN "MFG Name"
+F 5 "MBR0530T10G" H 1950 3450 60  0001 C CNN "MFG Part Num"
+F 6 "Diode Schottky/30V/500mA/SOD-123" H 1950 3450 60  0001 C CNN "Description"
 	1    1950 3450
 	-1   0    0    1
@@
 F 4 "Murata" H 1300 3750 60  0001 C CNN "MFG Name"
 F 5 "BLM18EG601SN1" H 1300 3750 60  0001 C CNN "MFG Part Num"
-F 6 "Bead/EMI supression" H 1300 3750 60  0001 C CNN "Description"
+F 6 "Inductor/Bead/0603" H 1300 3750 60  0001 C CNN "Description"
 	1    1300 3750
 	0    1    1    0
@@
 	1    0    0    -1
 $EndComp
-$Comp
-L LED D3
-U 1 1 547467CD
-P 7200 3650
-F 0 "D3" H 7200 3750 50  0000 C CNN
-F 1 "Blue_Led" H 7200 3550 50  0000 C CNN
-F 2 "0603" H 7200 3650 60  0001 C CNN
-F 3 "D" H 7200 3650 60  0001 C CNN
-F 4 "M" H 7200 3650 60  0001 C CNN "MFG Name"
-F 5 "P" H 7200 3650 60  0001 C CNN "MFG Part Num"
-F 6 "Led/Blue/0603" H 7200 3650 60  0001 C CNN "Description"
-	1    7200 3650
-	0    1    1    0
-$EndComp
 Text HLabel 9250 5350 1    45   Output ~ 0
 MAVLINK_GND
@@
 F 1 "22nH" V 7250 3200 40  0000 C CNN
 F 2 "0603" H 7150 3200 60  0001 C CNN
+F 3 "D" H 7150 3200 60  0001 C CNN
 F 4 "Samsung" H 7150 3200 60  0001 C CNN "MFG Name"
 F 5 "CIH10T22NJNC" H 7150 3200 60  0001 C CNN "MFG Part Num"
-F 6 "Inductor/22nH/0603" H 7150 3200 60  0001 C CNN "Description"
+F 6 "Inductor/22nH/+-10%/0.4R/0603" H 7150 3200 60  0001 C CNN "Description"
 	1    7150 3200
 	0    1    1    0
@@
 F 4 "Samsung" H 2650 3450 60  0001 C CNN "MFG Name"
 F 5 "CIH10T22NJNC" H 2650 3450 60  0001 C CNN "MFG Part Num"
-F 6 "Inductor/22nH/" H 2650 3450 60  0001 C CNN "Description"
+F 6 "Inductor/22nH/+-10%/0.4R/0603" H 2650 3450 60  0001 C CNN "Description"
 	1    2650 3450
 	0    1    1    0
@@
 F 4 "On Semiconductor" H 5350 4250 60  0001 C CNN "MFG Name"
 F 5 "MBR0530T1G" H 5350 4250 60  0001 C CNN "MFG Part Num"
-F 6 "Diode/Schottky/30V/0.5A/SOD-123" H 5350 4250 60  0001 C CNN "Description"
+F 6 "Diode/Schottky/30V/500mA/SOD-123" H 5350 4250 60  0001 C CNN "Description"
 	1    5350 4250
 	0    1    1    0
