File: air/osd/hardware/64_pin_lite/air_osd_v2_2/kicad_project/video_out.sch (KiCad schematic (older format))
At the start: 8 parts, among them P5 SIL5, U7 LM358DMR2G

Commit message: added Fiducials and settings to get pos file
Parts:
- C24, C25: MFG Name TDK Corporation -> M; MFG Part Num C2012X5R1A336M125AC -> P
- L7: value BLM18PG471SN1 -> BLM18EG601SN1; MFG Part Num BLM18PG471SN1 -> BLM18EG601SN1
Changed lines of the file:
@@
-EESchema Schematic File Version 2  date Thu 18 Jun 2015 19:52:51 BST
+EESchema Schematic File Version 2  date Fri 19 Jun 2015 22:46:51 BST
 LIBS:lm358
 LIBS:conn_6
@@
 LIBS:R0link
 LIBS:emi_filter
+LIBS:fiducial
+LIBS:osd-cache
 EELAYER 25  0
 EELAYER END
@@
 Sheet 7 8
 Title ""
-Date "18 jun 2015"
+Date "19 jun 2015"
 Rev ""
 Comp ""
@@
 P 7850 2650
 F 0 "L7" V 7800 2650 40  0000 C CNN
-F 1 "BLM18PG471SN1" V 7950 2650 40  0000 C CNN
+F 1 "BLM18EG601SN1" V 7950 2650 40  0000 C CNN
 F 2 "0603" H 7850 2650 60  0001 C CNN
 F 3 "search.murata.co.jp/Ceramy/image/img/PDF/ENG/L0110S0100BLM18P.pdf" H 7850 2650 60  0001 C CNN
 F 4 "Murata" H 7850 2650 60  0001 C CNN "MFG Name"
-F 5 "BLM18PG471SN1" H 7850 2650 60  0001 C CNN "MFG Part Num"
+F 5 "BLM18EG601SN1" H 7850 2650 60  0001 C CNN "MFG Part Num"
 F 6 "Inductor/0603" H 7850 2650 60  0001 C CNN "Description"
 	1    7850 2650
@@
 	4150 5600 4150 5950
 Wire Wire Line
-	4150 5950 3150 5950
-Wire Wire Line
-	3150 5950 3100 5950
+	4150 5950 3100 5950
 Wire Wire Line
 	3150 4950 3150 4900
 Wire Wire Line
-	8950 2750 9000 2750
-Wire Wire Line
-	9000 2750 9100 2750
+	8950 2750 9100 2750
 Wire Wire Line
 	9100 2550 8900 2550
@@
 	5750 3600 5600 3600
 Wire Wire Line
-	4700 3600 4800 3600
-Wire Wire Line
-	4800 3600 5200 3600
+	4700 3600 5200 3600
 Wire Wire Line
 	3700 3500 3300 3500
 Wire Wire Line
-	4700 2400 4800 2400
-Wire Wire Line
-	4800 2400 4950 2400
+	4700 2400 4950 2400
 Wire Wire Line
 	3400 2300 3700 2300
@@
 	9100 2650 8150 2650
 Wire Wire Line
-	6850 2650 7050 2650
-Wire Wire Line
-	7050 2650 7550 2650
+	6850 2650 7550 2650
 Wire Wire Line
 	3150 5850 3150 5950
 Wire Wire Line
-	3050 4900 3150 4900
-Wire Wire Line
-	3150 4900 4150 4900
+	3050 4900 4150 4900
 Wire Wire Line
 	4150 4900 4150 5200
@@
 F 2 "0805" H 5400 3600 60  0001 C CNN
 F 3 "D" H 5400 3600 60  0001 C CNN
-F 4 "TDK Corporation" H 5400 3600 60  0001 C CNN "MFG Name"
-F 5 "C2012X5R1A336M125AC" H 5400 3600 60  0001 C CNN "MFG Part Num"
+F 4 "M" H 5400 3600 60  0001 C CNN "MFG Name"
+F 5 "P" H 5400 3600 60  0001 C CNN "MFG Part Num"
 F 6 "Capacitor/33uF/10V/+-20%/X5R/0603" H 5400 3600 60  0001 C CNN "Description"
 	1    5400 3600
@@
 F 2 "0805" H 5350 2350 60  0001 C CNN
 F 3 "D" H 5350 2350 60  0001 C CNN
-F 4 "TDK Corporation" H 5350 2350 60  0001 C CNN "MFG Name"
-F 5 "C2012X5R1A336M125AC" H 5350 2350 60  0001 C CNN "MFG Part Num"
+F 4 "M" H 5350 2350 60  0001 C CNN "MFG Name"
+F 5 "P" H 5350 2350 60  0001 C CNN "MFG Part Num"
 F 6 "Capacitor/33uF/10V/+-20%/X5R/0805" H 5350 2350 60  0001 C CNN "Description"
 	1    5350 2350
