File: air/osd/hardware/64_pin_lite/air_osd_v2_2/kicad_project/video_out.sch (KiCad schematic (older format))
At the start: 8 parts, among them P5 SIL5, U7 LM358DMR2G

Commit message: changed diode pins side to comply with IPC-7351 2005 (dont have later spec)
Parts:
- C23: Description Capacitor/0.1uF/+-10%/X7R/0603 -> Capacitor/0.1uF/10V/+-10%/X7R/0603
Changed lines of the file:
@@
-EESchema Schematic File Version 2  date Sun 21 Jun 2015 14:24:06 BST
+EESchema Schematic File Version 2  date Thu 25 Jun 2015 08:05:44 BST
+LIBS:conn_20
+LIBS:conn_6
+LIBS:conn_5
+LIBS:conn_3
+LIBS:conn_2
 LIBS:power
 LIBS:device
@@
 LIBS:contrib
 LIBS:valves
+LIBS:diodesch_ipc7531_2005
 LIBS:osd-cache
 EELAYER 25  0
@@
 Sheet 7 8
 Title ""
-Date "20 jun 2015"
+Date "25 jun 2015"
 Rev ""
 Comp ""
@@
 F 4 "M" H 4150 5400 60  0001 C CNN "MFG Name"
 F 5 "P" H 4150 5400 60  0001 C CNN "MFG Part Num"
-F 6 "Capacitor/0.1uF/+-10%/X7R/0603" H 4150 5400 60  0001 C CNN "Description"
+F 6 "Capacitor/0.1uF/10V/+-10%/X7R/0603" H 4150 5400 60  0001 C CNN "Description"
 	1    4150 5400
 	1    0    0    -1

Commit message: v2.2 pcb hopefully ready to go
Parts:
- removed D5: MBR0530T1G, SOD-123, symbol DIODESCH
- added D5: MBR0530T1G, SOD-123, symbol DIODESCH_IPC7531_2005
- L7: Description Inductor/0603 -> Inductor/Bead/0603
Connections:
- net VIDEO_OUT_+V: now also D5.2 (An)
- net at C45.1, L7.2: now also D5.1 (Ca)
Changed lines of the file:
@@
-EESchema Schematic File Version 2  date Thu 25 Jun 2015 08:05:44 BST
+EESchema Schematic File Version 2  date Thu 25 Jun 2015 13:32:01 BST
 LIBS:conn_20
 LIBS:conn_6
@@
 LIBS:valves
 LIBS:diodesch_ipc7531_2005
+LIBS:led_ipc-7351_2005
 LIBS:osd-cache
 EELAYER 25  0
@@
 $EndDescr
 $Comp
+L DIODESCH_IPC7531_2005 D5
+U 1 1 558BBB81
+P 6650 2650
+F 0 "D5" H 6650 2750 40  0000 C CNN
+F 1 "MBR0530T1G" H 6650 2550 40  0000 C CNN
+F 2 "SOD-123" H 6650 2650 60  0001 C CNN
+F 3 "D" H 6650 2650 60  0001 C CNN
+F 4 "On Semiconductor" H 6650 2650 60  0001 C CNN "MFG Name"
+F 5 "MBR0530T1G" H 6650 2650 60  0001 C CNN "MFG Part Num"
+F 6 "Diode/Schottky/30V/500mA/SOD-123" H 6650 2650 60  0001 C CNN "Description"
+	1    6650 2650
+	-1   0    0    1
+$EndComp
+$Comp
 L INDUCTOR L7
 U 1 1 55828ED5
@@
 F 4 "Murata" H 7850 2650 60  0001 C CNN "MFG Name"
 F 5 "BLM18EG601SN1" H 7850 2650 60  0001 C CNN "MFG Part Num"
-F 6 "Inductor/0603" H 7850 2650 60  0001 C CNN "Description"
+F 6 "Inductor/Bead/0603" H 7850 2650 60  0001 C CNN "Description"
 	1    7850 2650
 	0    1    1    0
@@
 	4950 2400 4950 2350
 Wire Wire Line
-	6450 2650 6350 2650
+	6500 2650 6350 2650
 Wire Wire Line
 	9100 2650 8150 2650
 Wire Wire Line
-	6850 2650 7550 2650
+	6800 2650 7550 2650
 Wire Wire Line
 	3150 5850 3150 5950
@@
 	1    0    0    -1
 $EndComp
-$Comp
-L DIODESCH D5
-U 1 1 546F5AD9
-P 6650 2650
-F 0 "D5" H 6650 2750 40  0000 C CNN
-F 1 "MBR0530T1G" H 6650 2550 40  0000 C CNN
-F 2 "SOD-123" H 6650 2650 60  0001 C CNN
-F 3 "D" H 6650 2650 60  0001 C CNN
-F 4 "M" H 6650 2650 60  0001 C CNN "MFG Name"
-F 5 "P" H 6650 2650 60  0001 C CNN "MFG Part Num"
-F 6 "Diode/Schottky/30V/0.5A/SOD-123" H 6650 2650 60  0001 C CNN "Description"
-	1    6650 2650
-	1    0    0    -1
-$EndComp
