File: air/osd/hardware/64_pin_lite/air_osd_v2_2/kicad_project/camera.sch (KiCad schematic (older format))
At the start: 4 parts, among them K1 SIL3

Commit message: v2.2 pcb hopefully ready to go
Parts:
- removed D4: MBR0530T1G, SOD-123, symbol DIODESCH
- added D4: MBR0530T1G, SOD-123, symbol DIODESCH_IPC7531_2005
- L6: Description EMI Suppression filter -> Inductor/Bead/0603
Connections:
- net VIDEO_IN_+V: now also D4.2 (An)
- net at C39.1, L6.2: now also D4.1 (Ca)
Changed lines of the file:
@@
-EESchema Schematic File Version 2  date Thu 25 Jun 2015 08:05:44 BST
+EESchema Schematic File Version 2  date Thu 25 Jun 2015 13:32:01 BST
 LIBS:conn_20
 LIBS:conn_6
@@
 LIBS:valves
 LIBS:diodesch_ipc7531_2005
+LIBS:led_ipc-7351_2005
 LIBS:osd-cache
 EELAYER 25  0
@@
 $EndDescr
 $Comp
+L DIODESCH_IPC7531_2005 D4
+U 1 1 558BB778
+P 3250 3450
+F 0 "D4" H 3250 3550 40  0000 C CNN
+F 1 "MBR0530T1G" H 3250 3350 40  0000 C CNN
+F 2 "SOD-123" H 3250 3450 60  0001 C CNN
+F 3 "D" H 3250 3450 60  0001 C CNN
+F 4 "On Semiconductor" H 3250 3450 60  0001 C CNN "MFG Name"
+F 5 "MBR0530T1G" H 3250 3450 60  0001 C CNN "MFG Part Num"
+F 6 "Diode/Schottky/30V/500mA/SOD-123" H 3250 3450 60  0001 C CNN "Description"
+	1    3250 3450
+	-1   0    0    1
+$EndComp
+$Comp
 L INDUCTOR L6
 U 1 1 5582ABE4
@@
 F 4 "Murata" H 5100 3450 60  0001 C CNN "MFG Name"
 F 5 "BLM18EG601SN1" H 5100 3450 60  0001 C CNN "MFG Part Num"
-F 6 "EMI Suppression filter" H 5100 3450 60  0001 C CNN "Description"
+F 6 "Inductor/Bead/0603" H 5100 3450 60  0001 C CNN "Description"
 	1    5100 3450
 	0    1    1    0
@@
 	4050 4350 4050 4100
 Wire Wire Line
-	4800 3450 3450 3450
+	4800 3450 3400 3450
 Wire Wire Line
 	5400 3450 6950 3450
@@
 	6600 3550 6950 3550
 Wire Wire Line
-	3050 3450 2700 3450
+	3100 3450 2700 3450
 Wire Wire Line
 	4050 3700 4050 3450
@@
 Text HLabel 2700 3450 0    45   Input ~ 0
 VIDEO_IN_+V
-$Comp
-L DIODESCH D4
-U 1 1 546F5A7F
-P 3250 3450
-F 0 "D4" H 3250 3550 40  0000 C CNN
-F 1 "MBR0530T1G" H 3250 3350 40  0000 C CNN
-F 2 "SOD-123" H 3250 3450 60  0001 C CNN
-F 3 "www.onsemi.com/pub_link/Collateral/MBR0530T1-D.pdf" H 3250 3450 60  0001 C CNN
-F 4 "ON Semiconductor" H 3250 3450 60  0001 C CNN "MFG Name"
-F 5 "MBR0530T1G" H 3250 3450 60  0001 C CNN "MFG Part Num"
-F 6 "Diode/Schottky/30V/0.5A/SOD-123" H 3250 3450 60  0001 C CNN "Description"
-	1    3250 3450
-	1    0    0    -1
-$EndComp
 Text HLabel 6750 3350 0    45   Output ~ 0
 VIDEO_IN
