File: air/osd/hardware/64_pin_lite/air_osd_v2_2/kicad_project/mavlink_port.sch (KiCad schematic (older format))
At the start: 13 parts, among them P4 SIL6, U6 SI8642

Commit message: changed diode pins side to comply with IPC-7351 2005 (dont have later spec)
Parts:
- D7: value Red Led -> Red_Led
Changed lines of the file:
@@
-EESchema Schematic File Version 2  date Sun 21 Jun 2015 14:24:06 BST
+EESchema Schematic File Version 2  date Thu 25 Jun 2015 08:05:44 BST
+LIBS:conn_20
+LIBS:conn_6
+LIBS:conn_5
+LIBS:conn_3
+LIBS:conn_2
 LIBS:power
 LIBS:device
@@
 LIBS:contrib
 LIBS:valves
+LIBS:diodesch_ipc7531_2005
 LIBS:osd-cache
 EELAYER 25  0
@@
 Sheet 6 8
 Title ""
-Date "20 jun 2015"
+Date "25 jun 2015"
 Rev ""
 Comp ""
@@
 P 9100 1650
 F 0 "D7" H 9100 1750 50  0000 C CNN
-F 1 "Red Led" H 9100 1550 50  0000 C CNN
+F 1 "Red_Led" H 9100 1550 50  0000 C CNN
 F 2 "0603" H 9100 1650 60  0001 C CNN
 F 3 "D" H 9100 1650 60  0001 C CNN

Commit message: v2.2 pcb hopefully ready to go
Parts:
- removed D7: Red_Led, 0603, symbol LED
- added D7: Red_Led, 0603, symbol LED_IPC-7351_2005
Connections:
- net FC_+5V: now also D7.2 (An)
- net at R24.2: now also D7.1 (Ca)
Changed lines of the file:
@@
-EESchema Schematic File Version 2  date Thu 25 Jun 2015 08:05:44 BST
+EESchema Schematic File Version 2  date Thu 25 Jun 2015 13:32:01 BST
 LIBS:conn_20
 LIBS:conn_6
@@
 LIBS:valves
 LIBS:diodesch_ipc7531_2005
+LIBS:led_ipc-7351_2005
 LIBS:osd-cache
 EELAYER 25  0
@@
 Comment4 ""
 $EndDescr
+$Comp
+L LED_IPC-7351_2005 D7
+U 1 1 558BBFDE
+P 9100 1650
+F 0 "D7" H 9100 1450 50  0000 C CNN
+F 1 "Red_Led" H 9150 1900 50  0000 C CNN
+F 2 "0603" H 9100 1650 60  0001 C CNN
+F 3 "D" H 9100 1650 60  0001 C CNN
+F 4 "M" H 9100 1650 60  0001 C CNN "MFG Name"
+F 5 "P" H 9100 1650 60  0001 C CNN "MFG Part Num"
+F 6 "Led/Red/0603" H 9100 1650 60  0001 C CNN "Description"
+	1    9100 1650
+	0    -1   -1   0
+$EndComp
 Wire Wire Line
 	9350 1350 9100 1350
 Wire Wire Line
-	9100 1350 9100 1450
+	9100 1350 9100 1500
 Wire Wire Line
 	9100 2450 9100 2500
@@
 Connection ~ 7700 2000
 Wire Wire Line
-	9100 1950 9100 1850
+	9100 1950 9100 1800
 Text Label 9250 2500 0    45   ~ 0
 FC_GND
@@
 $EndComp
 $Comp
-L LED D7
-U 1 1 54FC3E4D
-P 9100 1650
-F 0 "D7" H 9100 1750 50  0000 C CNN
-F 1 "Red_Led" H 9100 1550 50  0000 C CNN
-F 2 "0603" H 9100 1650 60  0001 C CNN
-F 3 "D" H 9100 1650 60  0001 C CNN
-F 4 "M" H 9100 1650 60  0001 C CNN "MFG Name"
-F 5 "P" H 9100 1650 60  0001 C CNN "MFG Part Num"
-F 6 "Led/Red/0603" H 9100 1650 60  0001 C CNN "Description"
-	1    9100 1650
-	0    1    1    0
-$EndComp
-$Comp
