File: air/osd/hardware/64_pin_lite/air_osd_v2_2/kicad_project/mavlink_port.sch (KiCad schematic (older format))
At the start: 13 parts, among them P4 SIL6, U6 SI8642

Commit message: update scheatics for Kicad
Parts:
- C21, C22, C37, C38, C43: symbol C -> C-RESCUE-osd
- R24, R26, R27, R28, R29: symbol R -> R-RESCUE-osd
Changed lines of the file:
@@
-EESchema Schematic File Version 2  date Fri 26 Jun 2015 07:08:11 BST
+EESchema Schematic File Version 2
+LIBS:osd-rescue
 LIBS:conn_20
 LIBS:conn_6
@@
 LIBS:memory
 LIBS:xilinx
-LIBS:special
 LIBS:microcontrollers
 LIBS:dsp
@@
 LIBS:led_ipc-7351_2005
 LIBS:osd-cache
-EELAYER 25  0
+EELAYER 25 0
 EELAYER END
-$Descr A4 11700 8267
+$Descr A4 11693 8268
 encoding utf-8
 Sheet 6 8
@@
 FC_+5V
 $Comp
-L R R24
+L R-RESCUE-osd R24
 U 1 1 54FC3E86
 P 9100 2200
@@
 $EndComp
 $Comp
-L C C43
+L C-RESCUE-osd C43
 U 1 1 54FC3D3F
 P 7250 1650
@@
 $EndComp
 $Comp
-L C C37
+L C-RESCUE-osd C37
 U 1 1 547D825F
 P 6650 4600
@@
 $EndComp
 $Comp
-L C C38
+L C-RESCUE-osd C38
 U 1 1 547D8257
 P 7400 4600
@@
 $EndComp
 $Comp
-L R R29
+L R-RESCUE-osd R29
 U 1 1 547D81DE
 P 7750 3500
@@
 $EndComp
 $Comp
-L R R28
+L R-RESCUE-osd R28
 U 1 1 547D81C5
 P 7000 4250
@@
 $EndComp
 $Comp
-L R R27
+L R-RESCUE-osd R27
 U 1 1 547D816E
 P 6750 3400
@@
 $EndComp
 $Comp
-L R R26
+L R-RESCUE-osd R26
 U 1 1 547D813B
 P 6750 3150
@@
 FC_+5V
 $Comp
-L C C22
+L C-RESCUE-osd C22
 U 1 1 54734555
 P 7700 1650
@@
 F 1 "0.1uF" H 7750 1550 50  0000 L CNN
 F 2 "0603" H 7700 1650 60  0001 C CNN
+F 3 "" H 7700 1650 60  0001 C CNN
 F 4 "M" H 7700 1650 60  0001 C CNN "MFG Name"
 F 5 "P" H 7700 1650 60  0001 C CNN "MFG Part Num"
@@
 $EndComp
 $Comp
-L C C21
+L C-RESCUE-osd C21
 U 1 1 54734552
 P 2800 2550
@@
 F 1 "0.1uF" H 2850 2450 50  0000 L CNN
 F 2 "0603" H 2800 2550 60  0001 C CNN
+F 3 "" H 2800 2550 60  0001 C CNN
 F 4 "M" H 2800 2550 60  0001 C CNN "MFG Name"
 F 5 "P" H 2800 2550 60  0001 C CNN "MFG Part Num"
@@
 F 0 "#FLG05" H 8350 5020 30  0001 C CNN
 F 1 "PWR_FLAG" H 8350 4980 30  0000 C CNN
+F 2 "" H 8350 4750 60  0001 C CNN
+F 3 "" H 8350 4750 60  0001 C CNN
 	1    8350 4750
 	1    0    0    -1
@@
 F 0 "#FLG06" H 6700 2570 30  0001 C CNN
 F 1 "PWR_FLAG" H 6700 2530 30  0000 C CNN
+F 2 "" H 6700 2300 60  0001 C CNN
+F 3 "" H 6700 2300 60  0001 C CNN
 	1    6700 2300
 	1    0    0    -1
@@
 F 1 "SIL6" V 9550 3550 60  0000 C CNN
 F 2 "SIL6" H 9500 3550 60  0001 C CNN
+F 3 "" H 9500 3550 60  0001 C CNN
 F 4 "0.1 in pitch header/6 contacts" H 9500 3550 60  0001 C CNN "Description"
 	1    9500 3550
