File: air/osd/hardware/64_pin_lite/air_osd_v2_2/kicad_project/osd.sch (KiCad schematic (older format))
At the start: 6 parts

Commit message: changed diode pins side to comply with IPC-7351 2005 (dont have later spec)
Parts:
- FID1, FID2, FID3, FID4, FID5, FID6: footprint (none) -> FIDUCIAL; Description (none) -> fiducial; MFG Name (none) -> none; MFG Part Num (none) -> none
Changed lines of the file:
@@
-EESchema Schematic File Version 2  date Sun 21 Jun 2015 14:24:06 BST
+EESchema Schematic File Version 2  date Thu 25 Jun 2015 08:05:44 BST
+LIBS:conn_20
+LIBS:conn_6
+LIBS:conn_5
+LIBS:conn_3
+LIBS:conn_2
 LIBS:power
 LIBS:device
@@
 LIBS:contrib
 LIBS:valves
+LIBS:diodesch_ipc7531_2005
 LIBS:osd-cache
 EELAYER 25  0
@@
 Sheet 1 8
 Title ""
-Date "20 jun 2015"
+Date "25 jun 2015"
 Rev ""
 Comp ""
@@
 F 0 "FID6" H 9300 6350 60  0000 C CNN
 F 1 "FIDUCIAL" H 9250 6750 60  0000 C CNN
+F 2 "FIDUCIAL" H 9300 6550 60  0001 C CNN
+F 3 "none" H 9300 6550 60  0001 C CNN
+F 4 "none" H 9300 6550 60  0001 C CNN "MFG Name"
+F 5 "none" H 9300 6550 60  0001 C CNN "MFG Part Num"
+F 6 "fiducial" H 9300 6550 60  0001 C CNN "Description"
 	1    9300 6550
 	1    0    0    -1
@@
 F 0 "FID4" H 8450 6350 60  0000 C CNN
 F 1 "FIDUCIAL" H 8400 6750 60  0000 C CNN
+F 2 "FIDUCIAL" H 8450 6550 60  0001 C CNN
+F 3 "none" H 8450 6550 60  0001 C CNN
+F 4 "none" H 8450 6550 60  0001 C CNN "MFG Name"
+F 5 "none" H 8450 6550 60  0001 C CNN "MFG Part Num"
+F 6 "fiducial" H 8450 6550 60  0001 C CNN "Description"
 	1    8450 6550
 	1    0    0    -1
@@
 F 0 "FID2" H 7600 6300 60  0000 C CNN
 F 1 "FIDUCIAL" H 7550 6700 60  0000 C CNN
+F 2 "FIDUCIAL" H 7600 6500 60  0001 C CNN
+F 3 "none" H 7600 6500 60  0001 C CNN
+F 4 "none" H 7600 6500 60  0001 C CNN "MFG Name"
+F 5 "none" H 7600 6500 60  0001 C CNN "MFG Part Num"
+F 6 "fiducial" H 7600 6500 60  0001 C CNN "Description"
 	1    7600 6500
 	1    0    0    -1
@@
 F 0 "FID5" H 9250 5450 60  0000 C CNN
 F 1 "FIDUCIAL" H 9200 5850 60  0000 C CNN
+F 2 "FIDUCIAL" H 9250 5650 60  0001 C CNN
+F 3 "none" H 9250 5650 60  0001 C CNN
+F 4 "none" H 9250 5650 60  0001 C CNN "MFG Name"
+F 5 "none" H 9250 5650 60  0001 C CNN "MFG Part Num"
+F 6 "fiducial" H 9250 5650 60  0001 C CNN "Description"
 	1    9250 5650
 	1    0    0    -1
@@
 F 0 "FID3" H 8450 5450 60  0000 C CNN
 F 1 "FIDUCIAL" H 8400 5850 60  0000 C CNN
+F 2 "FIDUCIAL" H 8450 5650 60  0001 C CNN
+F 3 "none" H 8450 5650 60  0001 C CNN
+F 4 "none" H 8450 5650 60  0001 C CNN "MFG Name"
+F 5 "none" H 8450 5650 60  0001 C CNN "MFG Part Num"
+F 6 "fiducial" H 8450 5650 60  0001 C CNN "Description"
 	1    8450 5650
 	1    0    0    -1
@@
 F 0 "FID1" H 7600 5450 60  0000 C CNN
 F 1 "FIDUCIAL" H 7550 5850 60  0000 C CNN
+F 2 "FIDUCIAL" H 7600 5650 60  0001 C CNN
+F 3 "none" H 7600 5650 60  0001 C CNN
+F 4 "none" H 7600 5650 60  0001 C CNN "MFG Name"
+F 5 "none" H 7600 5650 60  0001 C CNN "MFG Part Num"
+F 6 "fiducial" H 7600 5650 60  0001 C CNN "Description"
 	1    7600 5650
 	1    0    0    -1
