File: air/osd/hardware/64_pin_lite/air_osd_v2_2/kicad_project/video_circuit.sch (KiCad schematic (older format))
At the start: 34 parts, among them P10 Pad, P12 Pad, P9 Pad, U10 FMS6141, U11 DAC084S085, U12 ADG704, U13 OPA830, U8 MCP6562, U9 TLV3501

Commit message: changed diode pins side to comply with IPC-7351 2005 (dont have later spec)
Parts:
- C26: Description Capacitor/0.1uF/+-10%/X7R/0603 -> Capacitor/0.1uF/10V/+-10%/X7R/0603
Changed lines of the file:
@@
-EESchema Schematic File Version 2  date Sun 21 Jun 2015 14:24:06 BST
+EESchema Schematic File Version 2  date Thu 25 Jun 2015 08:05:44 BST
+LIBS:conn_20
+LIBS:conn_6
+LIBS:conn_5
+LIBS:conn_3
+LIBS:conn_2
 LIBS:power
 LIBS:device
@@
 LIBS:contrib
 LIBS:valves
+LIBS:diodesch_ipc7531_2005
 LIBS:osd-cache
 EELAYER 25  0
@@
 Sheet 8 8
 Title ""
-Date "20 jun 2015"
+Date "25 jun 2015"
 Rev ""
 Comp ""
@@
 F 4 "M" H 1700 1600 60  0001 C CNN "MFG Name"
 F 5 "P" H 1700 1600 60  0001 C CNN "MFG Part Num"
-F 6 "Capacitor/0.1uF/+-10%/X7R/0603" H 1700 1600 60  0001 C CNN "Description"
+F 6 "Capacitor/0.1uF/10V/+-10%/X7R/0603" H 1700 1600 60  0001 C CNN "Description"
 	1    1700 1600
 	0    1    1    0
