File: air/osd/hardware/64_pin_lite/air_osd_v2_2/kicad_project/video_circuit.sch (KiCad schematic (older format))
At the start: 34 parts, among them P10 Pad, P12 Pad, P9 Pad, U10 FMS6141, U11 DAC084S085, U12 ADG704, U13 OPA830, U8 MCP6562, U9 TLV3501

Commit message: update scheatics for Kicad
Parts:
- C26, C27, C28, C29, C30, C31, C32, C33, C34, C35, C36, C44: symbol C -> C-RESCUE-osd
- R11, R12, R13, R14, R15, R16, R17, R18, R19, R20, R21, R22, R23: symbol R -> R-RESCUE-osd
Changed lines of the file:
@@
-EESchema Schematic File Version 2  date Fri 26 Jun 2015 07:08:11 BST
+EESchema Schematic File Version 2
+LIBS:osd-rescue
 LIBS:conn_20
 LIBS:conn_6
@@
 LIBS:memory
 LIBS:xilinx
-LIBS:special
 LIBS:microcontrollers
 LIBS:dsp
@@
 LIBS:led_ipc-7351_2005
 LIBS:osd-cache
-EELAYER 25  0
+EELAYER 25 0
 EELAYER END
-$Descr A4 11700 8267
+$Descr A4 11693 8268
 encoding utf-8
 Sheet 8 8
@@
 	4050 3250 1600 3250
 Wire Wire Line
-	4050 3250 4050 3500
+	4050 3500 4050 3250
 Wire Wire Line
 	1600 3250 1600 3950
@@
 	7600 5450 7600 5550
 $Comp
-L C C44
+L C-RESCUE-osd C44
 U 1 1 550014A9
 P 7600 5750
@@
 CSYNC
 $Comp
-L C C29
+L C-RESCUE-osd C29
 U 1 1 546DB5EF
 P 6950 5750
@@
 $EndComp
 $Comp
-L C C35
+L C-RESCUE-osd C35
 U 1 1 546DB5BD
 P 9600 5750
@@
 $EndComp
 $Comp
-L C C36
+L C-RESCUE-osd C36
 U 1 1 546DB542
 P 9900 5750
@@
 $EndComp
 $Comp
-L C C32
+L C-RESCUE-osd C32
 U 1 1 546DB404
 P 8700 5750
@@
 $EndComp
 $Comp
-L C C30
+L C-RESCUE-osd C30
 U 1 1 546DB398
 P 7250 5750
@@
 $EndComp
 $Comp
-L C C34
+L C-RESCUE-osd C34
 U 1 1 546DB394
 P 9300 5750
@@
 $EndComp
 $Comp
-L C C28
+L C-RESCUE-osd C28
 U 1 1 546DB366
 P 6650 5750
@@
 $EndComp
 $Comp
-L C C31
+L C-RESCUE-osd C31
 U 1 1 546DB339
 P 8400 5750
@@
 $EndComp
 $Comp
-L C C33
+L C-RESCUE-osd C33
 U 1 1 546DB332
 P 9000 5750
@@
 VIDEO_+5V
 $Comp
-L R R17
+L R-RESCUE-osd R17
 U 1 1 546B544B
 P 4500 4500
@@
 $EndComp
 $Comp
-L R R12
+L R-RESCUE-osd R12
 U 1 1 546B5003
 P 3200 3650
@@
 $EndComp
 $Comp
-L R R16
+L R-RESCUE-osd R16
 U 1 1 546B4FEB
 P 4450 3500
@@
 $EndComp
 $Comp
-L R R19
+L R-RESCUE-osd R19
 U 1 1 544D2243
 P 6050 6400
@@
 $EndComp
 $Comp
-L R R23
+L R-RESCUE-osd R23
 U 1 1 544CEF88
 P 10300 1600
@@
 VIDEO_SAMPLE
 $Comp
-L R R21
+L R-RESCUE-osd R21
 U 1 1 544A415B
 P 8800 1850
@@
 $EndComp
 $Comp
-L R R22
+L R-RESCUE-osd R22
 U 1 1 544A412C
 P 9450 2400
@@
 $EndComp
 $Comp
-L R R20
+L R-RESCUE-osd R20
 U 1 1 544A4107
 P 8450 1500
@@
 $EndComp
 $Comp
-L R R18
+L R-RESCUE-osd R18
 U 1 1 5448D75F
 P 5000 5550
@@
 GREY_D
 $Comp
-L R R15
+L R-RESCUE-osd R15
 U 1 1 5448BA29
 P 4200 6950
@@
 $EndComp
 $Comp
-L R R14
+L R-RESCUE-osd R14
 U 1 1 5448BA26
 P 4200 5800
@@
 $EndComp
 $Comp
-L C C27
+L C-RESCUE-osd C27
 U 1 1 5448B99E
 P 3650 6500
@@
 $EndComp
 $Comp
-L R R13
+L R-RESCUE-osd R13
 U 1 1 5448B6A1
 P 3300 6200
@@
 $EndComp
 $Comp
-L C C26
+L C-RESCUE-osd C26
 U 1 1 541E8561
 P 1700 1600
@@
 $EndComp
 $Comp
-L R R11
+L R-RESCUE-osd R11
 U 1 1 541E78CF
 P 1350 2150

Commit message: tracker v2 commit bundle
Parts:
- U8: symbol MCP6562 -> MCP6562-RESCUE-osd
Changed lines of the file:
@@
 Csync circuit
 $Comp
-L MCP6562 U8
+L MCP6562-RESCUE-osd U8
 U 3 1 54707205
 P 1750 7050
+AR Path="/54707205" Ref="U8"  Part="3"
+AR Path="/544A4CB8/54707205" Ref="U8"  Part="3"
 F 0 "U8" H 1800 7250 60  0000 L CNN
 F 1 "MCP6562" H 1700 6850 60  0000 L CNN
@@
 $EndComp
 $Comp
-L MCP6562 U8
+L MCP6562-RESCUE-osd U8
 U 2 1 54706BB6
 P 5200 6400
+AR Path="/54706BB6" Ref="U8"  Part="2"
+AR Path="/544A4CB8/54706BB6" Ref="U8"  Part="2"
 F 0 "U8" H 5250 6600 60  0000 L CNN
 F 1 "MCP6562" H 5150 6200 60  0000 L CNN
@@
 $EndComp
 $Comp
-L MCP6562 U8
+L MCP6562-RESCUE-osd U8
 U 1 1 54706B91
 P 2450 6200
+AR Path="/54706B91" Ref="U8"  Part="1"
+AR Path="/544A4CB8/54706B91" Ref="U8"  Part="1"
 F 0 "U8" H 2500 6400 60  0000 L CNN
 F 1 "MCP6562" H 2400 6000 60  0000 L CNN
