File: air/osd/hardware/64_pin_lite/air_osd_v2_2/kicad_project/expansion.sch (KiCad schematic (older format))
At the start: 5 parts, among them P11 SIL1, P2 SIL20, P3 SIL20

Commit message: update scheatics for Kicad
Parts:
- R25, R30: symbol R -> R-RESCUE-osd
Changed lines of the file:
@@
-EESchema Schematic File Version 2  date Fri 26 Jun 2015 07:08:11 BST
+EESchema Schematic File Version 2
+LIBS:osd-rescue
 LIBS:conn_20
 LIBS:conn_6
@@
 LIBS:memory
 LIBS:xilinx
-LIBS:special
 LIBS:microcontrollers
 LIBS:dsp
@@
 LIBS:led_ipc-7351_2005
 LIBS:osd-cache
-EELAYER 25  0
+EELAYER 25 0
 EELAYER END
-$Descr A4 11700 8267
+$Descr A4 11693 8268
 encoding utf-8
 Sheet 5 8
@@
 Connection ~ 4200 2550
 $Comp
-L R R30
+L R-RESCUE-osd R30
 U 1 1 5580AC4E
 P 4600 2150
@@
 $EndComp
 $Comp
-L R R25
+L R-RESCUE-osd R25
 U 1 1 5580AC49
 P 4600 1900
@@
 F 1 "SIL1" H 7300 2555 30  0001 C CNN
 F 2 "SIL1" H 7300 2500 60  0001 C CNN
+F 3 "" H 7300 2500 60  0001 C CNN
 F 4 "0.1 in pitch header/1 contact" H 7300 2500 60  0001 C CNN "Description"
 	1    7300 2500
@@
 F 0 "#FLG03" H 5550 2820 30  0001 C CNN
 F 1 "PWR_FLAG" H 5550 2780 30  0000 C CNN
+F 2 "" H 5550 2550 60  0001 C CNN
+F 3 "" H 5550 2550 60  0001 C CNN
 	1    5550 2550
 	1    0    0    -1
@@
 F 0 "#FLG04" H 6200 2620 30  0001 C CNN
 F 1 "PWR_FLAG" H 6200 2580 30  0000 C CNN
+F 2 "" H 6200 2350 60  0001 C CNN
+F 3 "" H 6200 2350 60  0001 C CNN
 	1    6200 2350
 	1    0    0    -1
@@
 F 1 "SIL20" V 3150 3500 60  0000 C CNN
 F 2 "SIL20" H 3100 3500 60  0001 C CNN
+F 3 "" H 3100 3500 60  0001 C CNN
 F 4 "0.1 in pitch header/20 contacts" H 3100 3500 60  0001 C CNN "Description"
 	1    3100 3500
@@
 F 1 "SIL20" V 7000 3450 60  0000 C CNN
 F 2 "SIL20" H 6950 3450 60  0001 C CNN
+F 3 "" H 6950 3450 60  0001 C CNN
 F 4 "0.1 in pitch header/20 contacts" H 6950 3450 60  0001 C CNN "Description"
 	1    6950 3450
