File: air/osd/hardware/air_osd_v3/kicad/video_circuit.sch (KiCad schematic (older format))
At the start: 29 parts, among them P10 Pad, P12 Pad, P9 Pad, U10 FMS6141, U8 MCP6562

Commit message: update scheatics for Kicad
Parts:
- removed Q?: FET_N, symbol FET_N
- added Q?: NPN, symbol NPN
- added R?: 10R, symbol R
- R?: value R -> 64.9R
- R?: value R -> 237R
- R?: value R -> 205R
- R?: value R -> 154R
Connections:
- net labels added: +3.3V
- net labels removed: +5V
- wire segments 115 -> 116

Commit message: update kicad files
Parts:
- C27, C28, C29, C31, C32, C33, C44, C?: symbol C -> C-RESCUE-osd
- R13, R14, R15, R18, R19, R? (x3): symbol R -> R-RESCUE-osd
- R?: value 64.9R -> ?; symbol R -> R-RESCUE-osd
- R?: value 237R -> ?; symbol R -> R-RESCUE-osd
- R?: value 205R -> ?; symbol R -> R-RESCUE-osd
- R?: value 154R -> ?; symbol R -> R-RESCUE-osd
- R?: value 10R -> ?; symbol R -> R-RESCUE-osd
- RV?: symbol POT -> POT-RESCUE-osd
Connections:
- wire segments 116 -> 87
Changed lines of the file:
@@
-EESchema Schematic File Version 2  date Wed 18 May 2016 11:24:51 BST
+EESchema Schematic File Version 2
+LIBS:osd-rescue
 LIBS:conn_20
 LIBS:conn_6
@@
 LIBS:memory
 LIBS:xilinx
-LIBS:special
 LIBS:microcontrollers
 LIBS:dsp
@@
 LIBS:bd9g101g
 LIBS:ld39015mxxr
-EELAYER 25  0
+LIBS:osd-cache
+EELAYER 25 0
 EELAYER END
-$Descr A4 11700 8267
+$Descr A4 11693 8268
 encoding utf-8
 Sheet 8 8
@@
 $EndDescr
 $Comp
-L +3.3V #PWR?
+L +3.3V-RESCUE-osd #PWR?
 U 1 1 573C42B3
 P 5250 2300
 F 0 "#PWR?" H 5250 2260 30  0001 C CNN
 F 1 "+3.3V" H 5250 2410 30  0000 C CNN
+F 2 "" H 5250 2300 60  0001 C CNN
+F 3 "" H 5250 2300 60  0001 C CNN
 	1    5250 2300
 	1    0    0    -1
@@
 	2100 2900 1900 2900
 Wire Wire Line
-	1900 3000 1900 2900
-Wire Wire Line
-	1900 2900 1900 2800
+	1900 2800 1900 3000
 Wire Wire Line
 	1600 3150 1600 3700
@@
 Connection ~ 3650 7000
 Wire Wire Line
-	3750 7000 3650 7000
-Wire Wire Line
-	3650 7000 1200 7000
+	1200 7000 3750 7000
 Connection ~ 1200 5550
 Wire Wire Line
-	4750 5550 4200 5550
-Wire Wire Line
-	4200 5550 1200 5550
+	1200 5550 4750 5550
 Connection ~ 1200 6350
 Wire Wire Line
@@
 Connection ~ 2950 1300
 Wire Wire Line
-	6750 1600 6750 1300
-Wire Wire Line
-	6750 1300 2950 1300
-Wire Wire Line
-	2950 1300 2800 1300
+	6750 1300 6750 1600
+Wire Wire Line
+	2800 1300 6750 1300
 Wire Wire Line
 	6200 2350 5500 2350
@@
 Connection ~ 5250 3000
 Wire Wire Line
-	4650 2000 3900 2000
-Wire Wire Line
-	3900 2000 3600 2000
-Wire Wire Line
-	7600 5550 7600 5450
-Wire Wire Line
-	7600 5450 6950 5450
-Wire Wire Line
-	6950 5450 6650 5450
-Wire Wire Line
-	6650 5450 6450 5450
+	3600 2000 4650 2000
+Wire Wire Line
+	7600 5450 7600 5550
+Wire Wire Line
+	6450 5450 7600 5450
 Connection ~ 3800 6200
 Wire Wire Line
@@
 Connection ~ 8700 5450
 Wire Wire Line
-	8700 5550 8700 5450
+	8700 5450 8700 5550
 Wire Wire Line
 	6650 5550 6650 5450
@@
 	8700 5950 8700 6250
 Wire Wire Line
-	8250 5450 8400 5450
-Wire Wire Line
-	8400 5450 8700 5450
-Wire Wire Line
-	8700 5450 9000 5450
-Wire Wire Line
-	3550 6200 3650 6200
-Wire Wire Line
-	3650 6200 3800 6200
-Wire Wire Line
-	3800 6200 3900 6200
+	8250 5450 9000 5450
+Wire Wire Line
+	3550 6200 3900 6200
 Connection ~ 3650 6200
 Wire Wire Line
@@
 	5250 5550 5700 5550
 Wire Wire Line
-	5700 5550 5700 5900
-Wire Wire Line
-	5700 5900 5700 6400
+	5700 5550 5700 6400
 Connection ~ 5700 6400
 Wire Wire Line
-	5600 6400 5700 6400
-Wire Wire Line
-	5700 6400 5800 6400
-Wire Wire Line
-	9000 6250 8700 6250
-Wire Wire Line
-	8700 6250 8400 6250
-Wire Wire Line
-	8400 6250 7850 6250
-Wire Wire Line
-	7850 6250 7600 6250
-Wire Wire Line
-	7600 6250 6950 6250
-Wire Wire Line
-	6950 6250 6650 6250
+	5600 6400 5800 6400
+Wire Wire Line
+	6650 6250 9000 6250
 Wire Wire Line
 	8400 6250 8400 5950
@@
 	2950 1550 2950 1300
 Wire Wire Line
-	1100 3700 1600 3700
-Wire Wire Line
-	1600 3700 1900 3700
-Wire Wire Line
-	1900 3700 2950 3700
+	1100 3700 2950 3700
 Wire Wire Line
 	2950 3700 2950 2450
@@
 Connection ~ 7600 6250
 Wire Wire Line
-	5250 3100 5250 3000
-Wire Wire Line
-	5250 3000 5250 2950
-Wire Wire Line
-	5250 2950 5250 2900
+	5250 2900 5250 3100
 Wire Wire Line
 	5250 2400 5250 2300
 Wire Wire Line
-	1600 2650 1600 2150
-Wire Wire Line
-	1600 2150 1600 2000
-Wire Wire Line
-	1300 2000 1600 2000
-Wire Wire Line
-	1600 2000 1900 2000
+	1600 2000 1600 2650
+Wire Wire Line
+	1300 2000 1900 2000
 Connection ~ 1600 2000
 Wire Wire Line
-	6200 2000 5800 2000
-Wire Wire Line
-	5800 2000 5150 2000
-Wire Wire Line
-	5150 3950 5250 3950
-Wire Wire Line
-	5250 3950 5800 3950
-Wire Wire Line
-	5800 3950 6750 3950
+	5150 2000 6200 2000
+Wire Wire Line
+	5150 3950 6750 3950
 Wire Wire Line
 	6750 3950 6750 2900
 Connection ~ 5250 3950
 Wire Wire Line
-	1200 6250 1200 6350
-Wire Wire Line
-	1200 6350 1200 6400
-Wire Wire Line
-	1200 5400 1200 5550
-Wire Wire Line
-	1200 5550 1200 5750
+	1200 6250 1200 6400
+Wire Wire Line
+	1200 5400 1200 5750
 Wire Wire Line
 	1200 7000 1200 6900
@@
 	5800 2450 5800 2000
 $Comp
-L R R?
+L R-RESCUE-osd R?
 U 1 1 573C2AD5
 P 5800 2700
 F 0 "R?" V 5880 2700 50  0000 C CNN
-F 1 "10R" V 5800 2700 50  0000 C CNN
+F 1 "?" V 5800 2700 50  0000 C CNN
+F 2 "" H 5800 2700 60  0001 C CNN
+F 3 "" H 5800 2700 60  0001 C CNN
 	1    5800 2700
 	1    0    0    -1
@@
 F 0 "Q?" H 5900 3150 50  0000 R CNN
 F 1 "NPN" H 5900 3450 50  0000 R CNN
+F 2 "" H 5900 3300 60  0001 C CNN
+F 3 "" H 5900 3300 60  0001 C CNN
 	1    5900 3300
 	-1   0    0    -1
@@
 MASK
 $Comp
-L R R?
+L R-RESCUE-osd R?
 U 1 1 5683A4DE
 P 1900 3250
 F 0 "R?" V 1980 3250 50  0000 C CNN
 F 1 "100R" V 1900 3250 50  0000 C CNN
+F 2 "" H 1900 3250 60  0001 C CNN
+F 3 "" H 1900 3250 60  0001 C CNN
 	1    1900 3250
 	1    0    0    -1
@@
 $EndComp
 $Comp
-L R R?
+L R-RESCUE-osd R?
 U 1 1 56799206
 P 1200 6650
 F 0 "R?" V 1280 6650 50  0000 C CNN
 F 1 "R" V 1200 6650 50  0000 C CNN
+F 2 "" H 1200 6650 60  0001 C CNN
+F 3 "" H 1200 6650 60  0001 C CNN
 	1    1200 6650
 	1    0    0    -1
@@
 F 0 "U?" H 6650 2150 60  0000 C CNN
 F 1 "TS5A3157" H 6400 1650 60  0000 C CNN
+F 2 "" H 6750 2250 60  0001 C CNN
+F 3 "" H 6750 2250 60  0001 C CNN
 	1    6750 2250
 	-1   0    0    -1
 $EndComp
 $Comp
-L C C?
+L C-RESCUE-osd C?
 U 1 1 56798F36
 P 2100 2000
 F 0 "C?" H 2150 2100 50  0000 L CNN
 F 1 "C" H 2150 1900 50  0000 L CNN
+F 2 "" H 2100 2000 60  0001 C CNN
+F 3 "" H 2100 2000 60  0001 C CNN
 	1    2100 2000
 	0    1    1    0
 $EndComp
 $Comp
-L R R?
+L R-RESCUE-osd R?
 U 1 1 56798EE3
 P 1600 2900
 F 0 "R?" V 1680 2900 50  0000 C CNN
 F 1 "150R" V 1600 2900 50  0000 C CNN
+F 2 "" H 1600 2900 60  0001 C CNN
+F 3 "" H 1600 2900 60  0001 C CNN
 	1    1600 2900
 	1    0    0    -1
@@
 VIDEO_GND
 $Comp
-L POT RV?
+L POT-RESCUE-osd RV?
 U 1 1 567989BB
 P 1900 2550
 F 0 "RV?" H 1900 2450 50  0000 C CNN
 F 1 "100R" H 1900 2550 50  0000 C CNN
+F 2 "" H 1900 2550 60  0001 C CNN
+F 3 "" H 1900 2550 60  0001 C CNN
 	1    1900 2550
 	0    1    1    0
@@
 VIDEO_GND
 $Comp
-L R R?
+L R-RESCUE-osd R?
 U 1 1 56798AD0
 P 4650 3000
 F 0 "R?" V 4730 3000 50  0000 C CNN
-F 1 "154R" V 4650 3000 50  0000 C CNN
+F 1 "?" V 4650 3000 50  0000 C CNN
+F 2 "" H 4650 3000 60  0001 C CNN
+F 3 "" H 4650 3000 60  0001 C CNN
 	1    4650 3000
 	0    1    1    0
 $EndComp
 $Comp
-L R R?
+L R-RESCUE-osd R?
 U 1 1 56798ACC
 P 5250 3350
 F 0 "R?" V 5330 3350 50  0000 C CNN
-F 1 "205R" V 5250 3350 50  0000 C CNN
+F 1 "?" V 5250 3350 50  0000 C CNN
+F 2 "" H 5250 3350 60  0001 C CNN
+F 3 "" H 5250 3350 60  0001 C CNN
 	1    5250 3350
 	1    0    0    -1
 $EndComp
 $Comp
-L R R?
+L R-RESCUE-osd R?
 U 1 1 56798AC8
 P 5250 2650
 F 0 "R?" V 5330 2650 50  0000 C CNN
-F 1 "237R" V 5250 2650 50  0000 C CNN
+F 1 "?" V 5250 2650 50  0000 C CNN
+F 2 "" H 5250 2650 60  0001 C CNN
+F 3 "" H 5250 2650 60  0001 C CNN
 	1    5250 2650
 	1    0    0    -1
 $EndComp
 $Comp
-L R R?
+L R-RESCUE-osd R?
 U 1 1 56798A1D
 P 4900 2000
 F 0 "R?" V 4980 2000 50  0000 C CNN
-F 1 "64.9R" V 4900 2000 50  0000 C CNN
+F 1 "?" V 4900 2000 50  0000 C CNN
+F 2 "" H 4900 2000 60  0001 C CNN
+F 3 "" H 4900 2000 60  0001 C CNN
 	1    4900 2000
 	0    1    1    0
 $EndComp
 $Comp
-L C C44
+L C-RESCUE-osd C44
 U 1 1 550014A9
 P 7600 5750
@@
 CSYNC
 $Comp
-L C C29
+L C-RESCUE-osd C29
 U 1 1 546DB5EF
 P 6950 5750
@@
 $EndComp
 $Comp
-L C C32
+L C-RESCUE-osd C32
 U 1 1 546DB404
 P 8700 5750
@@
 $EndComp
 $Comp
-L C C28
+L C-RESCUE-osd C28
 U 1 1 546DB366
 P 6650 5750
@@
 $EndComp
 $Comp
-L C C31
+L C-RESCUE-osd C31
 U 1 1 546DB339
 P 8400 5750
@@
 $EndComp
 $Comp
-L C C33
+L C-RESCUE-osd C33
 U 1 1 546DB332
 P 9000 5750
@@
 VIDEO_+5V
 $Comp
-L R R19
+L R-RESCUE-osd R19
 U 1 1 544D2243
 P 6050 6400
@@
 VIDEO_SAMPLE
 $Comp
-L R R18
+L R-RESCUE-osd R18
 U 1 1 5448D75F
 P 5000 5550
@@
 $EndComp
 $Comp
-L R R15
+L R-RESCUE-osd R15
 U 1 1 5448BA29
 P 1200 6000
@@
 $EndComp
 $Comp
-L R R14
+L R-RESCUE-osd R14
 U 1 1 5448BA26
 P 1200 5150
@@
 $EndComp
 $Comp
-L C C27
+L C-RESCUE-osd C27
 U 1 1 5448B99E
 P 3650 6500
@@
 $EndComp
 $Comp
-L R R13
+L R-RESCUE-osd R13
 U 1 1 5448B6A1
 P 3300 6200
