File: air/osd/hardware/air_osd_v3/kicad/camera.sch (KiCad schematic (older format))
At the start: 4 parts, among them K1 SIL3

Commit message: update kicad files
Parts:
- C39: symbol C -> C-RESCUE-osd
Changed lines of the file:
@@
-EESchema Schematic File Version 2  date Wed 18 May 2016 11:24:51 BST
+EESchema Schematic File Version 2
+LIBS:osd-rescue
 LIBS:conn_20
 LIBS:conn_6
@@
 LIBS:memory
 LIBS:xilinx
-LIBS:special
 LIBS:microcontrollers
 LIBS:dsp
@@
 LIBS:bd9g101g
 LIBS:ld39015mxxr
-EELAYER 25  0
+LIBS:osd-cache
+EELAYER 25 0
 EELAYER END
-$Descr A4 11700 8267
+$Descr A4 11693 8268
 encoding utf-8
 Sheet 4 8
@@
 Connection ~ 4050 3450
 $Comp
-L C C39
+L C-RESCUE-osd C39
 U 1 1 5580ACEA
 P 4050 3900
@@
 F 1 "SIL3" V 7350 3450 40  0000 C CNN
 F 2 "SIL3" H 7300 3450 60  0001 C CNN
+F 3 "" H 7300 3450 60  0001 C CNN
 F 4 "0.1 in pitch header connector/3 contacts" H 7300 3450 60  0001 C CNN "Description"
 	1    7300 3450
