File: air/osd/hardware/air_osd_v3/kicad/mcu.sch (KiCad schematic (older format))
At the start: 29 parts, among them P1 SIL2, P6 Pad, P7 Pad, P8 Pad, U1 SI501, U2 STM32F405RGT6, U3 74LVC1G86

Commit message: update kicad files
Parts:
- C1, C10, C2, C4, C5, C7, C8: symbol C -> C-RESCUE-osd
- C11, C3, C6, C9: symbol CP1 -> CP1-RESCUE-osd
- R1, R2, R3, R31, R32, R4, R5, R6, R7: symbol R -> R-RESCUE-osd
Changed lines of the file:
@@
-EESchema Schematic File Version 2  date Wed 18 May 2016 11:24:51 BST
+EESchema Schematic File Version 2
+LIBS:osd-rescue
 LIBS:conn_20
 LIBS:conn_6
@@
 LIBS:memory
 LIBS:xilinx
-LIBS:special
 LIBS:microcontrollers
 LIBS:dsp
@@
 LIBS:bd9g101g
 LIBS:ld39015mxxr
-EELAYER 25  0
+LIBS:osd-cache
+EELAYER 25 0
 EELAYER END
-$Descr A4 11700 8267
+$Descr A4 11693 8268
 encoding utf-8
 Sheet 2 8
@@
 MCU_+3.3V
 $Comp
-L R R32
+L R-RESCUE-osd R32
 U 1 1 55814873
 P 9350 4650
@@
 $EndComp
 $Comp
-L R R31
+L R-RESCUE-osd R31
 U 1 1 55814870
 P 9050 4650
@@
 MCU_+3.3V
 $Comp
-L R R3
+L R-RESCUE-osd R3
 U 1 1 54734401
 P 7925 1900
@@
 Prog  Jumper
 $Comp
-L R R7
+L R-RESCUE-osd R7
 U 1 1 54734400
 P 10450 2800
@@
 MCU_GND
 $Comp
-L C C10
+L C-RESCUE-osd C10
 U 1 1 547343FF
 P 10450 3400
@@
 F 1 "SIL2" V 8425 1075 40  0000 C CNN
 F 2 "SIL2" H 8375 1075 60  0001 C CNN
+F 3 "" H 8375 1075 60  0001 C CNN
 F 4 "0.1 in pitch header/2 contacts" H 8375 1075 60  0001 C CNN "Description"
 	1    8375 1075
@@
 MCU_GND
 $Comp
-L C C1
+L C-RESCUE-osd C1
 U 1 1 5470A326
 P 1450 2975
@@
 $EndComp
 $Comp
-L CP1 C11
+L CP1-RESCUE-osd C11
 U 1 1 5470A08D
 P 8975 6325
@@
 $EndComp
 $Comp
-L R R1
+L R-RESCUE-osd R1
 U 1 1 546F4821
 P 5100 6175
@@
 HEARTBEAT_LED
 $Comp
-L R R2
+L R-RESCUE-osd R2
 U 1 1 546E5ED3
 P 6650 1100
@@
 MCU_VDDA
 $Comp
-L C C2
+L C-RESCUE-osd C2
 U 1 1 546CA664
 P 2425 6500
@@
 AV_TELEM_TXO
 $Comp
-L R R4
+L R-RESCUE-osd R4
 U 1 1 546B3A56
 P 9800 5225
@@
 RAW_FRSKY_TXO
 $Comp
-L R R5
+L R-RESCUE-osd R5
 U 1 1 546A8268
 P 9825 5000
@@
 MAVLINK_TXO
 $Comp
-L R R6
+L R-RESCUE-osd R6
 U 1 1 54676508
 P 9825 5550
@@
 AV_DAC_CLK
 $Comp
-L CP1 C3
+L CP1-RESCUE-osd C3
 U 1 1 543A7664
 P 5550 7200
@@
 $EndComp
 $Comp
-L CP1 C6
+L CP1-RESCUE-osd C6
 U 1 1 543A7660
 P 8950 3100
@@
 $EndComp
 $Comp
-L CP1 C9
+L CP1-RESCUE-osd C9
 U 1 1 543A7353
 P 8650 6325
@@
 $EndComp
 $Comp
-L C C8
+L C-RESCUE-osd C8
 U 1 1 543A72F3
 P 8250 6325
@@
 $EndComp
 $Comp
-L C C7
+L C-RESCUE-osd C7
 U 1 1 543A72EF
 P 7900 6325
@@
 $EndComp
 $Comp
-L C C5
+L C-RESCUE-osd C5
 U 1 1 543A72EC
 P 7550 6325
@@
 $EndComp
 $Comp
-L C C4
+L C-RESCUE-osd C4
 U 1 1 543A72BA
 P 7200 6325
