File: air/osd/hardware/air_osd_v3/kicad/psu.sch (KiCad schematic (older format))
At the start: 19 parts, among them U4 BD9G101G, U5 LD39015MXXR

Commit message: update kicad files
Parts:
- C13, C14, C15, C17, C18, C19, C20, C40, C42: symbol C -> C-RESCUE-osd
- R10, R8, R9: symbol R -> R-RESCUE-osd
- U5: symbol LD39015MXXR -> LD39015MxxR
Changed lines of the file:
@@
-EESchema Schematic File Version 2  date Wed 18 May 2016 11:24:51 BST
+EESchema Schematic File Version 2
+LIBS:osd-rescue
 LIBS:conn_20
 LIBS:conn_6
@@
 LIBS:memory
 LIBS:xilinx
-LIBS:special
 LIBS:microcontrollers
 LIBS:dsp
@@
 LIBS:bd9g101g
 LIBS:ld39015mxxr
-EELAYER 25  0
+LIBS:osd-cache
+EELAYER 25 0
 EELAYER END
-$Descr A4 11700 8267
+$Descr A4 11693 8268
 encoding utf-8
 Sheet 3 8
@@
 SWITCHER_CB
 $Comp
-L C C42
+L C-RESCUE-osd C42
 U 1 1 54F874D2
 P 1700 4000
@@
 F 0 "#FLG01" H 7600 3320 30  0001 C CNN
 F 1 "PWR_FLAG" H 7600 3280 30  0000 C CNN
+F 2 "" H 7600 3050 60  0001 C CNN
+F 3 "" H 7600 3050 60  0001 C CNN
 	1    7600 3050
 	1    0    0    -1
@@
 HUB_GND
 $Comp
-L C C40
+L C-RESCUE-osd C40
 U 1 1 54846E5A
 P 2650 4100
@@
 $EndComp
 $Comp
-L C C20
+L C-RESCUE-osd C20
 U 1 1 54749249
 P 9950 4200
@@
 $EndComp
 $Comp
-L C C19
+L C-RESCUE-osd C19
 U 1 1 547491F8
 P 9550 4200
@@
 MCU_+3.3V
 $Comp
-L LD39015MXXR U5
+L LD39015MxxR U5
 U 1 1 5474880F
 P 8850 3900
@@
 $EndComp
 $Comp
-L C C18
+L C-RESCUE-osd C18
 U 1 1 5474880E
 P 7950 4150
@@
 $EndComp
 $Comp
-L R R10
+L R-RESCUE-osd R10
 U 1 1 547467E3
 P 7200 4200
@@
 $EndComp
 $Comp
-L C C15
+L C-RESCUE-osd C15
 U 1 1 5472ED3C
 P 6450 3550
@@
 F 0 "#FLG02" H 3000 3520 30  0001 C CNN
 F 1 "PWR_FLAG" H 3000 3480 30  0000 C CNN
+F 2 "" H 3000 3250 60  0001 C CNN
+F 3 "" H 3000 3250 60  0001 C CNN
 	1    3000 3250
 	1    0    0    -1
 $EndComp
 $Comp
-L C C17
+L C-RESCUE-osd C17
 U 1 1 54711603
 P 7550 4250
@@
 $EndComp
 $Comp
-L R R8
+L R-RESCUE-osd R8
 U 1 1 5433B3C9
 P 6150 3550
@@
 $EndComp
 $Comp
-L R R9
+L R-RESCUE-osd R9
 U 1 1 5433B3C8
 P 6150 4250
@@
 $EndComp
 $Comp
-L C C14
+L C-RESCUE-osd C14
 U 1 1 5433B3C6
 P 5150 3500
@@
 $EndComp
 $Comp
-L C C13
+L C-RESCUE-osd C13
 U 1 1 5433B3C5
 P 3300 4100
