File: air/osd/hardware/air_osd_v3/kicad/video_out.sch (KiCad schematic (older format))
At the start: 8 parts, among them P5 SIL5, U7 LM358DMR2G

Commit message: update kicad files
Parts:
- C23, C24, C25, C45: symbol C -> C-RESCUE-osd
- U7: symbol LM358 -> LM358-RESCUE-osd
Changed lines of the file:
@@
-EESchema Schematic File Version 2  date Wed 18 May 2016 11:24:51 BST
+EESchema Schematic File Version 2
+LIBS:osd-rescue
 LIBS:conn_20
 LIBS:conn_6
@@
 LIBS:memory
 LIBS:xilinx
-LIBS:special
 LIBS:microcontrollers
 LIBS:dsp
@@
 LIBS:bd9g101g
 LIBS:ld39015mxxr
-EELAYER 25  0
+LIBS:osd-cache
+EELAYER 25 0
 EELAYER END
-$Descr A4 11700 8267
+$Descr A4 11693 8268
 encoding utf-8
 Sheet 7 8
@@
 Connection ~ 7050 2650
 $Comp
-L C C45
+L C-RESCUE-osd C45
 U 1 1 5580B0E2
 P 7050 2950
@@
 BUF_DAC_OUT1
 $Comp
-L C C25
+L C-RESCUE-osd C25
 U 1 1 5474951D
 P 5400 3600
@@
 $EndComp
 $Comp
-L C C24
+L C-RESCUE-osd C24
 U 1 1 54749516
 P 5350 2350
@@
 $EndComp
 $Comp
-L C C23
+L C-RESCUE-osd C23
 U 1 1 5470A75F
 P 4150 5400
@@
 VIDEO_OUT_+5V
 $Comp
-L LM358 U7
+L LM358-RESCUE-osd U7
 U 3 1 5470A57E
 P 3250 5400
@@
 F 1 "SIL5" V 9550 2550 50  0000 C CNN
 F 2 "SIL5" H 9500 2550 60  0001 C CNN
+F 3 "" H 9500 2550 60  0001 C CNN
 F 4 "0.1 in pitch header/5 contacts" H 9500 2550 60  0001 C CNN "Description"
 	1    9500 2550
@@
 VIDEO_OUT
 $Comp
-L LM358 U?
+L LM358-RESCUE-osd U?
 U 1 1 54675F35
 P 4200 3600
@@
 RAW_DAC_OUT2
 $Comp
-L LM358 U7
+L LM358-RESCUE-osd U7
 U 2 1 54675AC5
 P 4200 2400
