File: air/osd/hardware/sensor_board/hack_version/air_osd_module.sch (KiCad schematic (older format))
At the start: 66 parts

Commit message: update hack version to later kicad
Parts:
- C? (x6): symbol C -> C-RESCUE-flight_controller
- C?: symbol CP1 -> CP1-RESCUE-flight_controller
- D? (x2): symbol LED -> LED-RESCUE-flight_controller
- M?: symbol OSD_V2_1 -> OSD_v2_1
- R? (x33): symbol R -> R-RESCUE-flight_controller
