File: air/osd/hardware/sensor_board/hack_version/flight_controller.sch (KiCad schematic (older format))
At the start: 70 parts

Commit message: just update version info of the kicad flight controller schematic and lib, but no real chanes there
Other:
- note added: "(USART1)"
- note added: "(USART3)"
Changed lines of the file:
@@
-EESchema Schematic File Version 2  date Sat 24 Oct 2015 18:57:25 BST
+EESchema Schematic File Version 2  date Tue 17 Nov 2015 11:47:50 GMT
 LIBS:spst
 LIBS:power
@@
 Sheet 1 1
 Title ""
-Date "24 oct 2015"
+Date "17 nov 2015"
 Rev ""
 Comp ""
@@
 Comment4 ""
 $EndDescr
+Text Notes 6100 5300 0    60   ~ 0
+(USART3)
+Text Notes 6000 6150 0    60   ~ 0
+(USART1)
 Connection ~ 3150 1450
 Wire Wire Line

Commit message: add labels of usarts etc
Other:
- note added: "(SBUS_OUT)"
Changed lines of the file:
@@
-EESchema Schematic File Version 2  date Tue 17 Nov 2015 11:47:50 GMT
+EESchema Schematic File Version 2  date Thu 10 Dec 2015 12:45:17 GMT
 LIBS:spst
 LIBS:power
@@
 Sheet 1 1
 Title ""
-Date "17 nov 2015"
+Date "10 dec 2015"
 Rev ""
 Comp ""
@@
 Comment4 ""
 $EndDescr
+Text Notes 8500 3450 0    60   ~ 0
+(SBUS_OUT)
 Text Notes 6100 5300 0    60   ~ 0
 (USART3)

Commit message: some work on the FC
Parts:
- removed 22nH (x4): INDUCTOR, symbol INDUCTOR
- removed C? (x3): 10nF, symbol C
- removed C?: 0u1, symbol C
- removed C?: 100pF, symbol C
- removed C? (x2): C, symbol C
- removed C?: 4.7uF, symbol CP1
- removed D? (x2): LED, symbol LED
- removed K? (x7): CONN_3, symbol CONN_3
- removed M?: AIR_OSD_V2_2_PCB, symbol OSD_V2_1
- removed P?: BARO, symbol CONN_4
- removed P?: MAG, symbol CONN_4
- removed P?: CONN_5, symbol CONN_5
- removed P?: GPS, symbol CONN_4
- removed P?: MPU6000, symbol CONN_7
- removed P?: CONSOLE, symbol CONN_4
- removed P?: TELEM, symbol CONN_4
- removed Q? (x2): BS108, symbol FET_N
- removed R? (x2): 470R, symbol R
- removed R? (x2): 100R, symbol R
- removed R?: 1k, symbol R
- removed R?: 17K, symbol R
- removed R? (x2): 4.7K, symbol R
- removed R? (x4): 150R, symbol R
- removed R? (x8): 47R, symbol R
- removed R? (x8): R, symbol R
- removed R? (x2): 33K, symbol R
- removed R? (x2): 1K, symbol R
- removed R?: 300K, symbol R
- removed SW?: SPST, symbol SPST
- removed U? (x4): 74HCT125, symbol 74LS125
- removed U?: 74LVC1G86, symbol 74LVC1G86
Connections:
- net labels removed: +3.3V, +5V, 5V_3A, ADC_RSSI, AIR_SPD, AUX_ADC, BARO_SCL, BARO_SDA, BAT_I, BAT_V, EXTI1, EXTI2, FC_RX_GPS, FC_TX_GPS, FC_TX_RC, FRAM_NCS, GND, LED2, LED3, MAG_SCL, MAG_SDA, PPM_SUM, RAW_ASPD, RAW_PPMSUM, RAW_RC_OUT1, RAW_RC_OUT2, RAW_RC_OUT3, RAW_RC_OUT4, RAW_RSSI, RAW_SCL, RAW_SDA, RC_OUT1, RC_OUT2, RC_OUT3, RC_OUT4, SPI1_CK, SPI1_MISO, SPI1_MOSI, SPI_NCS, TELEM_RX, TELEM_TX, UART4_RX, UART4_TX, UART5_TX, VIN+
- wire segments 208 -> 0
- no-connect marks 2 -> 0
Other:
- note removed: "(SBUS_OUT)"
- note removed: "(USART1)"
- note removed: "(USART3)"
- note removed: "Analog airspeed sensor \nconnector"
- note removed: "Barometer should be\nIC on the board"
- note removed: "Console can also be used \nfor programming the board"
- note removed: "External mag\n connector"
- note removed: "Filter is used to prevent MCU \nswitching noise travelling to GPS\n(Port is isolated)\nA one chip solution may be better\n"
- note removed: "JTAG should still work\neven with LED's attached\n(not tested)"
- note removed: "Leds are done this way so that \nthe JTAG will still work"
- note removed: "MPU should be an\n IC on the board"
- note removed: "RC receiver connector\nbased on FrSKY D4-RII\nwith PPM_SUM, RSSI\nand Telemetry"
- note removed: "RCoutput shown give 4 outputs at up to 400Hz pulse referesh\nAdd the ADCAUX1 and ADCAUX2 outputs ass address select by the\nServo outputs. They can be used to provide\n16 RC outputs at 50 Hz pulse refresh with 4 2 to 4 line decoders and inverters"
- note removed: "SPI1_MOSI"
- note removed: "SPI1_SCK"
- note removed: "Solder jumper\nTo invert\nFrSKY TX out"
- note removed: "reset\nbutton"
