File: air/osd/hardware/sensor_board/hack_version/mpu6000.sch (KiCad schematic (older format))
At the start: 5 parts

Commit message: update hack version to later kicad
Parts:
- C? (x3): symbol C -> C-RESCUE-flight_controller
Changed lines of the file:
@@
-EESchema Schematic File Version 2  date Fri 08 Jan 2016 14:31:29 GMT
+EESchema Schematic File Version 2
+LIBS:flight_controller-rescue
 LIBS:spst
 LIBS:power
@@
 LIBS:fm25v01
 LIBS:flight_controller-cache
-EELAYER 25  0
+EELAYER 25 0
 EELAYER END
-$Descr A4 11700 8267
+$Descr A4 11693 8268
 encoding utf-8
 Sheet 3 5
@@
 	4400 3050 4400 3200
 $Comp
-L GND #PWR?
+L GND-RESCUE-flight_controller #PWR?
 U 1 1 568FBAAE
 P 6550 4600
 F 0 "#PWR?" H 6550 4600 30  0001 C CNN
 F 1 "GND" H 6550 4530 30  0001 C CNN
+F 2 "" H 6550 4600 60  0001 C CNN
+F 3 "" H 6550 4600 60  0001 C CNN
 	1    6550 4600
 	1    0    0    -1
 $EndComp
 $Comp
-L GND #PWR?
+L GND-RESCUE-flight_controller #PWR?
 U 1 1 568FBA40
 P 4400 3200
 F 0 "#PWR?" H 4400 3200 30  0001 C CNN
 F 1 "GND" H 4400 3130 30  0001 C CNN
+F 2 "" H 4400 3200 60  0001 C CNN
+F 3 "" H 4400 3200 60  0001 C CNN
 	1    4400 3200
 	1    0    0    -1
 $EndComp
 $Comp
-L GND #PWR?
+L GND-RESCUE-flight_controller #PWR?
 U 1 1 568FB8B6
 P 6100 5100
 F 0 "#PWR?" H 6100 5100 30  0001 C CNN
 F 1 "GND" H 6100 5030 30  0001 C CNN
+F 2 "" H 6100 5100 60  0001 C CNN
+F 3 "" H 6100 5100 60  0001 C CNN
 	1    6100 5100
 	1    0    0    -1
 $EndComp
 $Comp
-L C C?
+L C-RESCUE-flight_controller C?
 U 1 1 568FB8A6
 P 6100 4700
 F 0 "C?" H 6150 4800 50  0000 L CNN
 F 1 "C" H 6150 4600 50  0000 L CNN
+F 2 "" H 6100 4700 60  0001 C CNN
+F 3 "" H 6100 4700 60  0001 C CNN
 	1    6100 4700
 	1    0    0    -1
 $EndComp
 $Comp
-L GND #PWR?
+L GND-RESCUE-flight_controller #PWR?
 U 1 1 568FB852
 P 6500 1850
 F 0 "#PWR?" H 6500 1850 30  0001 C CNN
 F 1 "GND" H 6500 1780 30  0001 C CNN
+F 2 "" H 6500 1850 60  0001 C CNN
+F 3 "" H 6500 1850 60  0001 C CNN
 	1    6500 1850
 	1    0    0    -1
 $EndComp
 $Comp
-L C C?
+L C-RESCUE-flight_controller C?
 U 1 1 568FB843
 P 6200 2000
 F 0 "C?" H 6250 2100 50  0000 L CNN
 F 1 "C" H 6250 1900 50  0000 L CNN
+F 2 "" H 6200 2000 60  0001 C CNN
+F 3 "" H 6200 2000 60  0001 C CNN
 	1    6200 2000
 	1    0    0    -1
@@
 MPU600_NCS
 $Comp
-L GND #PWR?
+L GND-RESCUE-flight_controller #PWR?
 U 1 1 568FB2A7
 P 7350 3100
 F 0 "#PWR?" H 7350 3100 30  0001 C CNN
 F 1 "GND" H 7350 3030 30  0001 C CNN
+F 2 "" H 7350 3100 60  0001 C CNN
+F 3 "" H 7350 3100 60  0001 C CNN
 	1    7350 3100
 	1    0    0    -1
@@
 MPU6000_DIN
 $Comp
-L GND #PWR?
+L GND-RESCUE-flight_controller #PWR?
 U 1 1 568FA5D7
 P 7400 4250
 F 0 "#PWR?" H 7400 4250 30  0001 C CNN
 F 1 "GND" H 7400 4180 30  0001 C CNN
+F 2 "" H 7400 4250 60  0001 C CNN
+F 3 "" H 7400 4250 60  0001 C CNN
 	1    7400 4250
 	1    0    0    -1
 $EndComp
 $Comp
-L C C?
+L C-RESCUE-flight_controller C?
 U 1 1 568FA5C0
 P 7400 3800
 F 0 "C?" H 7450 3900 50  0000 L CNN
 F 1 "C" H 7450 3700 50  0000 L CNN
+F 2 "" H 7400 3800 60  0001 C CNN
+F 3 "" H 7400 3800 60  0001 C CNN
 	1    7400 3800
 	1    0    0    -1
@@
 F 0 "L?" V 7750 3550 40  0000 C CNN
 F 1 "INDUCTOR" V 7900 3550 40  0000 C CNN
+F 2 "" H 7800 3550 60  0001 C CNN
+F 3 "" H 7800 3550 60  0001 C CNN
 	1    7800 3550
 	0    1    1    0
@@
 F 0 "U?" H 6050 3300 60  0000 C CNN
 F 1 "MPU6000" H 6050 3300 60  0000 C CNN
+F 2 "" H 6050 3300 60  0001 C CNN
+F 3 "" H 6050 3300 60  0001 C CNN
 	1    6050 3300
 	1    0    0    -1
