File: ground/tracker/v1/hardware/using_quantracker_osd/tracker.sch (KiCad schematic (older format))
At the start: 33 parts, among them K1 CONN_3, K2 CONN_3, K3 CONN_3, M1 OSD_v2_2, P1 CONN_4, P2 CONN_4, P3 CONN_2, P4 CONN_5, SW1 SW_PUSH

Commit message: update tracker schematic
Connections:
- net TILT_PWM: now also M1.33 (PA11); no longer M1.44 (PB9)
Other:
- note added: "TIM1_CH4"
- note removed: "PPM_SUM"
- moved on the sheet: C9
Changed lines of the file:
@@
 LIBS:conn_8
 LIBS:cap3t
-LIBS:si8621
 LIBS:74aup2g240
 LIBS:tlcfilt
@@
 	10500 3200 10650 3200
 Wire Wire Line
-	6650 4325 7050 4325
+	6650 4325 7500 4325
 $Comp
 L TLCFILT LC2
@@
 L CAP3T C9
 U 1 1 58806F69
-P 7300 4325
-F 0 "C9" H 7450 4075 60  0000 C CNN
-F 1 "NFM18PS105R0J3" H 7525 4550 60  0000 C CNN
-F 2 "" H 7300 4325 60  0001 C CNN
-F 3 "" H 7300 4325 60  0001 C CNN
-	1    7300 4325
-	1    0    0    -1
-$EndComp
-Wire Wire Line
-	7550 4325 8000 4325
+P 7750 4325
+F 0 "C9" H 7900 4075 60  0000 C CNN
+F 1 "NFM18PS105R0J3" H 7975 4550 60  0000 C CNN
+F 2 "" H 7750 4325 60  0001 C CNN
+F 3 "" H 7750 4325 60  0001 C CNN
+	1    7750 4325
+	1    0    0    -1
+$EndComp
+Wire Wire Line
+	8000 4325 8175 4325
 Wire Wire Line
 	1525 3600 1300 3600
@@
 	7150 4525 7150 4675
 Wire Wire Line
-	7150 4675 7800 4675
-Wire Wire Line
-	7300 4675 7300 4525
+	7150 4675 7975 4675
+Wire Wire Line
+	7750 4675 7750 4525
 Wire Wire Line
 	4025 3625 4700 3625
 Wire Wire Line
 	4025 3625 4025 3425
-Connection ~ 7300 4675
+Connection ~ 7750 4675
 Wire Wire Line
 	6200 2300 8625 2300
@@
 Wire Wire Line
 	10125 2300 10325 2300
-Text Label 6775 3025 0    39   ~ 0
+Text Label 6800 4125 0    39   ~ 0
 TILT_PWM
-Wire Wire Line
-	6775 3025 6650 3025
 Text Label 2775 4125 0    60   ~ 0
 TILT_PWM
@@
 Text Label 6800 3925 0    60   ~ 0
 GND
-Text Label 7800 4675 0    60   ~ 0
+Text Label 7975 4675 0    60   ~ 0
 GND
 Text Label 3025 3225 2    60   ~ 0
 +5V
-Text Label 8000 4325 0    60   ~ 0
+Text Label 8175 4325 0    60   ~ 0
 +3.3V
 Text Label 1300 3600 2    60   ~ 0
@@
 NoConn ~ 6650 3825
 NoConn ~ 6650 4025
-NoConn ~ 6650 4125
 NoConn ~ 6650 4225
 NoConn ~ 6650 4425
@@
 L PWR_FLAG #FLG03
 U 1 1 5881E873
-P 6900 4300
-F 0 "#FLG03" H 6900 4395 50  0001 C CNN
-F 1 "PWR_FLAG" H 6900 4480 50  0000 C CNN
-F 2 "" H 6900 4300 50  0000 C CNN
-F 3 "" H 6900 4300 50  0000 C CNN
-	1    6900 4300
-	1    0    0    -1
-$EndComp
-Wire Wire Line
-	6900 4300 6900 4325
-Connection ~ 6900 4325
+P 7400 3850
+F 0 "#FLG03" H 7400 3945 50  0001 C CNN
+F 1 "PWR_FLAG" H 7400 4030 50  0000 C CNN
+F 2 "" H 7400 3850 50  0000 C CNN
+F 3 "" H 7400 3850 50  0000 C CNN
+	1    7400 3850
+	1    0    0    -1
+$EndComp
 $Comp
 L PWR_FLAG #FLG04
@@
 L PWR_FLAG #FLG05
 U 1 1 5881FB17
-P 7925 3950
-F 0 "#FLG05" H 7925 4045 50  0001 C CNN
-F 1 "PWR_FLAG" H 7925 4130 50  0000 C CNN
-F 2 "" H 7925 3950 50  0000 C CNN
-F 3 "" H 7925 3950 50  0000 C CNN
-	1    7925 3950
-	1    0    0    -1
-$EndComp
-Wire Wire Line
-	7925 3950 7925 4325
+P 8100 3950
+F 0 "#FLG05" H 8100 4045 50  0001 C CNN
+F 1 "PWR_FLAG" H 8100 4130 50  0000 C CNN
+F 2 "" H 8100 3950 50  0000 C CNN
+F 3 "" H 8100 3950 50  0000 C CNN
+	1    8100 3950
+	1    0    0    -1
+$EndComp
+Wire Wire Line
+	8100 3950 8100 4325
 Wire Wire Line
 	6800 3325 6650 3325
@@
 	4850 1975 4850 2200
 Connection ~ 4850 2200
-Connection ~ 7925 4325
+Connection ~ 8100 4325
 $Comp
 L PWR_FLAG #FLG06
@@
 MOTOR_I
 Text Notes 6000 4150 0    40   ~ 0
-PPM_SUM
+TIM1_CH4
 Text Notes 6025 4250 0    40   ~ 0
 SPI_NCS
@@
 Text Label 1975 7550 2    60   ~ 0
 PAN_GND
+Wire Wire Line
+	7400 3850 7400 4325
+Connection ~ 7400 4325
+Wire Wire Line
+	6650 4125 6800 4125
+NoConn ~ 6650 3025
 $EndSCHEMATC
